File: Ferinixie Fun Panel.kicad_pcb (KiCad board)
At the start: 2 copper layers, 110 x 75 mm, 37 parts, among them Q1 MMBT2222A, Q2 MMBT2222A, Q3 MMBT2222A, Q4 MMBT2222A, U1 HV5122_Flat, U3 RP2040-Tiny, U4 NCH8200HV, U5 OKI-78SR-5_1.5-W36H-C

Commit message: Saving before I restart
Parts:
- removed ? (x2): , 
- removed the REF** at (205.0, 98.5)
- removed the REF** at (213.5, 112.0)
- removed the REF** at (213.5, 45.0)
- added C4: 1uF, Capacitor_SMD:C_1206_3216Metric, F.Cu at (192.2, 176.2)
- added C5: 1uF, Capacitor_SMD:C_1206_3216Metric, F.Cu at (192.2, 179.6)
- added NE10: INS-1, NixFootprints:INS-1, F.Cu at (147.7, 196.3)
- added NE11: INS-1, NixFootprints:INS-1, F.Cu at (147.7, 205.4)
- added NE12: INS-1, NixFootprints:INS-1, F.Cu at (147.7, 214.6)
- added NE13: INS-1, NixFootprints:INS-1, F.Cu at (156.8, 169.1)
- added NE14: INS-1, NixFootprints:INS-1, F.Cu at (156.8, 178.2)
- added NE15: INS-1, NixFootprints:INS-1, F.Cu at (156.8, 187.2)
- added NE16: INS-1, NixFootprints:INS-1, F.Cu at (156.8, 196.3)
- added NE17: INS-1, NixFootprints:INS-1, F.Cu at (156.8, 205.4)
- added NE18: INS-1, NixFootprints:INS-1, F.Cu at (156.8, 214.6)
- added NE3: INS-1, NixFootprints:INS-1, F.Cu at (138.6, 187.2)
- added NE4: INS-1, NixFootprints:INS-1, F.Cu at (138.6, 196.3)
- added NE5: INS-1, NixFootprints:INS-1, F.Cu at (138.6, 205.4)
- added NE6: INS-1, NixFootprints:INS-1, F.Cu at (138.6, 214.6)
- added NE7: INS-1, NixFootprints:INS-1, F.Cu at (147.7, 169.1)
- added NE8: INS-1, NixFootprints:INS-1, F.Cu at (147.7, 178.2)
- added NE9: INS-1, NixFootprints:INS-1, F.Cu at (147.7, 187.2)
- added NIX1: IN-15A, NixFootprints:IN-15A Stepped, F.Cu at (121.0, 75.0)
- added NIX10: IN-15A, NixFootprints:IN-15A Stepped, F.Cu at (37.0, 106.0)
- added NIX11: IN-15A, NixFootprints:IN-15A Stepped, F.Cu at (121.0, 137.0)
- added NIX12: IN-15A, NixFootprints:IN-15A Stepped, F.Cu at (100.0, 137.0)
- added NIX13: IN-15A, NixFootprints:IN-15A Stepped, F.Cu at (79.0, 137.0)
- added NIX14: IN-15A, NixFootprints:IN-15A Stepped, F.Cu at (58.0, 137.0)
- added NIX15: IN-15A, NixFootprints:IN-15A Stepped, F.Cu at (37.0, 137.0)
- added NIX2: IN-15A, NixFootprints:IN-15A Stepped, F.Cu at (100.0, 75.0)
- added NIX3: IN-15A, NixFootprints:IN-15A Stepped, F.Cu at (79.0, 75.0)
- added NIX4: IN-15A, NixFootprints:IN-15A Stepped, F.Cu at (58.0, 75.0)
- added NIX8: IN-15A, NixFootprints:IN-15A Stepped, F.Cu at (79.0, 106.0)
- added NIX9: IN-15A, NixFootprints:IN-15A Stepped, F.Cu at (58.0, 106.0)
- added Q5: MMBT2222A, Package_TO_SOT_SMD:SOT-23, B.Cu at (201.5, 49.5)
- added Q6: MMBTA92, Package_TO_SOT_SMD:SOT-23, B.Cu at (134.6, 107.0)
- added Q7: MMBTA92, Package_TO_SOT_SMD:SOT-23, B.Cu at (138.0, 103.6)
- added Q8: MMBTA92, Package_TO_SOT_SMD:SOT-23, B.Cu at (141.5, 103.6)
- added Q9: MMBTA92, Package_TO_SOT_SMD:SOT-23, B.Cu at (145.0, 103.6)
- added R17: 100K, Resistor_SMD:R_1206_3216Metric, B.Cu at (96.0, 125.5)
- added R18: 100K, Resistor_SMD:R_1206_3216Metric, B.Cu at (75.0, 125.5)
- added R19: 100K, Resistor_SMD:R_1206_3216Metric, B.Cu at (54.0, 125.5)
- added R20: 100K, Resistor_SMD:R_1206_3216Metric, B.Cu at (33.0, 125.5)
- added R21: 100K, Resistor_SMD:R_1206_3216Metric, F.Cu at (169.7, 195.9)
- added R22: 100K, Resistor_SMD:R_1206_3216Metric, F.Cu at (169.7, 199.3)
- added R23: 100K, Resistor_SMD:R_1206_3216Metric, F.Cu at (175.3, 166.2)
- added R24: 10K, Resistor_SMD:R_1206_3216Metric, F.Cu at (175.3, 169.5)
- added R25: 20K, Resistor_SMD:R_1206_3216Metric, F.Cu at (175.3, 172.8)
- added R26: 100K, Resistor_SMD:R_1206_3216Metric, F.Cu at (175.3, 176.1)
- added R27: 100K, Resistor_SMD:R_1206_3216Metric, F.Cu at (175.3, 179.4)
- added R28: 100K, Resistor_SMD:R_1206_3216Metric, F.Cu at (175.3, 182.7)
- added R29: 100K, Resistor_SMD:R_1206_3216Metric, F.Cu at (175.3, 186.0)
- added R30: 100K, Resistor_SMD:R_1206_3216Metric, F.Cu at (175.3, 189.3)
- added R31: 100K, Resistor_SMD:R_1206_3216Metric, F.Cu at (175.3, 192.6)
- added R32: 100K, Resistor_SMD:R_1206_3216Metric, F.Cu at (175.3, 195.9)
- added R33: 100K, Resistor_SMD:R_1206_3216Metric, F.Cu at (175.3, 199.3)
- added R34: 100K, Resistor_SMD:R_1206_3216Metric, F.Cu at (180.9, 166.2)
- added R35: 100K, Resistor_SMD:R_1206_3216Metric, F.Cu at (180.9, 169.5)
- added R36: 20K, Resistor_SMD:R_1206_3216Metric, F.Cu at (180.9, 172.8)
- added R37: 100K, Resistor_SMD:R_1206_3216Metric, F.Cu at (180.9, 176.1)
- added R38: 100K, Resistor_SMD:R_1206_3216Metric, F.Cu at (180.9, 179.4)
- added R39: 100K, Resistor_SMD:R_1206_3216Metric, F.Cu at (180.9, 182.7)
- added R40: 20K, Resistor_SMD:R_1206_3216Metric, F.Cu at (180.9, 186.0)
- added R41: 10K, Resistor_SMD:R_1206_3216Metric, F.Cu at (180.9, 189.3)
- added R42: 20K, Resistor_SMD:R_1206_3216Metric, F.Cu at (180.9, 192.6)
- added R43: 20K, Resistor_SMD:R_1206_3216Metric, F.Cu at (180.9, 195.9)
- added R44: 20K, Resistor_SMD:R_1206_3216Metric, F.Cu at (180.9, 199.3)
- added R45: 10K, Resistor_SMD:R_1206_3216Metric, F.Cu at (186.5, 166.2)
- added R46: 20K, Resistor_SMD:R_1206_3216Metric, F.Cu at (186.5, 169.5)
- added R47: 20K, Resistor_SMD:R_1206_3216Metric, F.Cu at (186.5, 172.8)
- added R48: 20K, Resistor_SMD:R_1206_3216Metric, F.Cu at (186.5, 176.1)
- added R49: 10K, Resistor_SMD:R_1206_3216Metric, F.Cu at (186.5, 179.4)
- added R50: 20K, Resistor_SMD:R_1206_3216Metric, F.Cu at (186.5, 182.7)
- added R51: 20K, Resistor_SMD:R_1206_3216Metric, F.Cu at (186.5, 186.0)
- added R6: 10K, Resistor_SMD:R_1206_3216Metric, B.Cu at (117.0, 63.5)
- added R7: 10K, Resistor_SMD:R_1206_3216Metric, B.Cu at (96.0, 63.5)
- added R8: 10K, Resistor_SMD:R_1206_3216Metric, B.Cu at (75.0, 63.5)
- added REF**: PinHeader_1x10_P1.00mm_Vertical, Connector_PinHeader_1.00mm:PinHeader_1x10_P1.00mm_Vertical, F.Cu at (218.0, 106.0)
- added REF**: PinHeader_1x10_P1.00mm_Vertical, Connector_PinHeader_1.00mm:PinHeader_1x10_P1.00mm_Vertical, F.Cu at (197.0, 137.0)
- added REF**: PinHeader_1x10_P1.00mm_Vertical, Connector_PinHeader_1.00mm:PinHeader_1x10_P1.00mm_Vertical, F.Cu at (121.0, 75.0)
- added REF**: PinHeader_1x10_P1.00mm_Vertical, Connector_PinHeader_1.00mm:PinHeader_1x10_P1.00mm_Vertical, F.Cu at (239.0, 137.0)
- added REF**: PinHeader_1x10_P1.00mm_Vertical, Connector_PinHeader_1.00mm:PinHeader_1x10_P1.00mm_Vertical, F.Cu at (176.0, 75.0)
- added REF**: MountingHole_2.2mm_M2_DIN965_Pad, MountingHole:MountingHole_2.2mm_M2_DIN965_Pad, F.Cu at (253.5, 155.5)
- added REF**: PinHeader_1x10_P1.00mm_Vertical, Connector_PinHeader_1.00mm:PinHeader_1x10_P1.00mm_Vertical, F.Cu at (58.0, 106.0)
- added REF**: MountingHole_2.2mm_M2_DIN965_Pad, MountingHole:MountingHole_2.2mm_M2_DIN965_Pad, F.Cu at (140.5, 47.5)
- added REF**: MountingHole_2.2mm_M2_DIN965_Pad, MountingHole:MountingHole_2.2mm_M2_DIN965_Pad, F.Cu at (135.5, 155.5)
- added REF**: PinHeader_1x10_P1.00mm_Vertical, Connector_PinHeader_1.00mm:PinHeader_1x10_P1.00mm_Vertical, F.Cu at (37.0, 75.0)
- added REF**: PinHeader_1x10_P1.00mm_Vertical, Connector_PinHeader_1.00mm:PinHeader_1x10_P1.00mm_Vertical, F.Cu at (100.0, 106.0)
- added REF**: PinHeader_1x10_P1.00mm_Vertical, Connector_PinHeader_1.00mm:PinHeader_1x10_P1.00mm_Vertical, F.Cu at (155.0, 75.0)
- added REF**: PinHeader_1x10_P1.00mm_Vertical, Connector_PinHeader_1.00mm:PinHeader_1x10_P1.00mm_Vertical, F.Cu at (197.0, 106.0)
- added REF**: PinHeader_1x10_P1.00mm_Vertical, Connector_PinHeader_1.00mm:PinHeader_1x10_P1.00mm_Vertical, F.Cu at (121.0, 137.0)
- added REF**: PinHeader_1x10_P1.00mm_Vertical, Connector_PinHeader_1.00mm:PinHeader_1x10_P1.00mm_Vertical, F.Cu at (176.0, 137.0)
- added REF**: MountingHole_2.2mm_M2_DIN965_Pad, MountingHole:MountingHole_2.2mm_M2_DIN965_Pad, F.Cu at (22.5, 155.5)
- added REF**: PinHeader_1x10_P1.00mm_Vertical, Connector_PinHeader_1.00mm:PinHeader_1x10_P1.00mm_Vertical, F.Cu at (155.0, 106.0)
- added REF**: PinHeader_1x10_P1.00mm_Vertical, Connector_PinHeader_1.00mm:PinHeader_1x10_P1.00mm_Vertical, F.Cu at (239.0, 106.0)
- added REF**: PinHeader_1x10_P1.00mm_Vertical, Connector_PinHeader_1.00mm:PinHeader_1x10_P1.00mm_Vertical, F.Cu at (79.0, 106.0)
- added REF**: PinHeader_1x10_P1.00mm_Vertical, Connector_PinHeader_1.00mm:PinHeader_1x10_P1.00mm_Vertical, F.Cu at (37.0, 106.0)
- added REF**: PinHeader_1x10_P1.00mm_Vertical, Connector_PinHeader_1.00mm:PinHeader_1x10_P1.00mm_Vertical, F.Cu at (58.0, 75.0)
- added REF**: PinHeader_1x10_P1.00mm_Vertical, Connector_PinHeader_1.00mm:PinHeader_1x10_P1.00mm_Vertical, F.Cu at (37.0, 137.0)
- added REF**: MountingHole_2.2mm_M2_DIN965_Pad, MountingHole:MountingHole_2.2mm_M2_DIN965_Pad, F.Cu at (22.5, 47.5)
- added REF**: MountingHole_2.2mm_M2_DIN965_Pad, MountingHole:MountingHole_2.2mm_M2_DIN965_Pad, F.Cu at (253.5, 47.5)
- added REF**: PinHeader_1x10_P1.00mm_Vertical, Connector_PinHeader_1.00mm:PinHeader_1x10_P1.00mm_Vertical, F.Cu at (239.0, 75.0)
- added REF**: PinHeader_1x10_P1.00mm_Vertical, Connector_PinHeader_1.00mm:PinHeader_1x10_P1.00mm_Vertical, F.Cu at (100.0, 75.0)
- added REF**: PinHeader_1x10_P1.00mm_Vertical, Connector_PinHeader_1.00mm:PinHeader_1x10_P1.00mm_Vertical, F.Cu at (176.0, 106.0)
- added REF**: PinHeader_1x10_P1.00mm_Vertical, Connector_PinHeader_1.00mm:PinHeader_1x10_P1.00mm_Vertical, F.Cu at (197.0, 75.0)
- added REF**: PinHeader_1x10_P1.00mm_Vertical, Connector_PinHeader_1.00mm:PinHeader_1x10_P1.00mm_Vertical, F.Cu at (155.0, 137.0)
- added REF**: PinHeader_1x10_P1.00mm_Vertical, Connector_PinHeader_1.00mm:PinHeader_1x10_P1.00mm_Vertical, F.Cu at (79.0, 75.0)
- added REF**: MountingHole_2.2mm_M2_DIN965_Pad, MountingHole:MountingHole_2.2mm_M2_DIN965_Pad, F.Cu at (135.5, 47.5)
- added REF**: PinHeader_1x10_P1.00mm_Vertical, Connector_PinHeader_1.00mm:PinHeader_1x10_P1.00mm_Vertical, F.Cu at (218.0, 137.0)
- added REF**: PinHeader_1x10_P1.00mm_Vertical, Connector_PinHeader_1.00mm:PinHeader_1x10_P1.00mm_Vertical, F.Cu at (58.0, 137.0)
- added REF**: PinHeader_1x10_P1.00mm_Vertical, Connector_PinHeader_1.00mm:PinHeader_1x10_P1.00mm_Vertical, F.Cu at (100.0, 137.0)
- added REF**: MountingHole_2.2mm_M2_DIN965_Pad, MountingHole:MountingHole_2.2mm_M2_DIN965_Pad, F.Cu at (140.5, 155.5)
- added REF**: PinHeader_1x10_P1.00mm_Vertical, Connector_PinHeader_1.00mm:PinHeader_1x10_P1.00mm_Vertical, F.Cu at (79.0, 137.0)
- added REF**: PinHeader_1x10_P1.00mm_Vertical, Connector_PinHeader_1.00mm:PinHeader_1x10_P1.00mm_Vertical, F.Cu at (218.0, 75.0)
- added REF**: PinHeader_1x10_P1.00mm_Vertical, Connector_PinHeader_1.00mm:PinHeader_1x10_P1.00mm_Vertical, F.Cu at (121.0, 106.0)
- added U2: RP2040-Tiny, NixFootprints:RP2040-Tiny Package Extra Clearance SMD, F.Cu at (156.0, 56.5)
- C1, C2, Q1, Q2, Q4: moved to B.Cu
- Q3: value MMBT2222A -> MMBTA92; moved to B.Cu
- R1: value 100K -> 10K
- R10, R11: value 1K -> 10K; moved to B.Cu
- R12, R9: value 1K -> 20K; moved to B.Cu
- R13, R15, R16: value 10K -> 100K; moved to B.Cu
- R14: value 10K -> 20K; moved to B.Cu
- R2: value 100K -> 20K
- R3, R4, R5: value 20K -> 10K
- U1: value HV5122_Flat -> OKI-78SR-5_1.5-W36H-C; footprint Package_QFP:PQFP-44_10x10mm_P0.8mm -> Converter_DCDC:Converter_DCDC_Murata_OKI-78SR_Vertical
- U3: value RP2040-Tiny -> HV5122_Flat; footprint NixFootprints:RP2040-Tiny Package Extra Clearance SMD -> Package_QFP:PQFP-44_10x10mm_P0.8mm; moved to B.Cu
- U5: value OKI-78SR-5_1.5-W36H-C -> HV5122_Flat; footprint Converter_DCDC:Converter_DCDC_Murata_OKI-78SR_Vertical -> Package_QFP:PQFP-44_10x10mm_P0.8mm; moved to B.Cu
- moved U4 174.1 mm to (164.7, 225.0), turned to 0 degrees
- moved NIX5 146.5 mm to (37.0, 75.0)
- moved R15 135.8 mm to (33.0, 94.5), turned to 90 degrees
- moved G*** 135.6 mm to (68.8, 40.2)
- moved G*** 135.6 mm to (68.8, 27.8)
- moved C6 130.7 mm to (192.2, 182.9), turned to 0 degrees
- moved R14 120.7 mm to (54.0, 94.5), turned to 90 degrees
- moved R10 119.1 mm to (33.0, 63.5), turned to 90 degrees
- moved R5 116.0 mm to (164.1, 179.4), turned to 0 degrees
- moved R4 109.7 mm to (164.1, 176.1), turned to 0 degrees
- moved C3 109.4 mm to (192.2, 172.9), turned to 0 degrees
- moved R3 107.4 mm to (164.1, 172.8), turned to 0 degrees
- moved R13 106.4 mm to (75.0, 94.5), turned to 90 degrees
- moved NE1 103.8 mm to (138.6, 169.1), turned to 0 degrees
- moved R9 98.0 mm to (54.0, 63.5), turned to 90 degrees
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Connections:
- C3 pad 2: +170V -> +12V
- NIX5 pad 10: Net-(NIX5-%) -> Net-(NIX11-%)
- NIX5 pad 11: Net-(NIX5-n) -> Net-(NIX11-n)
- NIX5 pad 2: Net-(NIX5-µ) -> Net-(NIX11-µ)
- NIX5 pad 3: Net-(NIX5-P) -> Net-(NIX11-P)
- NIX5 pad 4: Net-(NIX5--) -> Net-(NIX11--)
- NIX5 pad 5: Net-(NIX5-+) -> Net-(NIX11-+)
- NIX5 pad 6: Net-(NIX5-m) -> Net-(NIX11-m)
- NIX5 pad 7: Net-(NIX5-M) -> Net-(NIX11-M)
- NIX5 pad 8: Net-(NIX5-k) -> Net-(NIX11-k)
- NIX5 pad 9: Net-(NIX5-П) -> Net-(NIX11-П)
- NIX6 pad 10: Net-(NIX6-%) -> Net-(NIX12-%)
- NIX6 pad 11: Net-(NIX6-n) -> Net-(NIX12-n)
- NIX6 pad 2: Net-(NIX6-µ) -> Net-(NIX12-µ)
- NIX6 pad 3: Net-(NIX6-P) -> Net-(NIX12-P)
- NIX6 pad 4: Net-(NIX6--) -> Net-(NIX12--)
- NIX6 pad 5: Net-(NIX6-+) -> Net-(NIX12-+)
- NIX6 pad 6: Net-(NIX6-m) -> Net-(NIX12-m)
- NIX6 pad 7: Net-(NIX6-M) -> Net-(NIX12-M)
- NIX6 pad 8: Net-(NIX6-k) -> Net-(NIX12-k)
- NIX6 pad 9: Net-(NIX6-П) -> Net-(NIX12-П)
- NIX7 pad 10: Net-(NIX7-%) -> Net-(NIX1-%)
- NIX7 pad 11: Net-(NIX7-n) -> Net-(NIX1-n)
- NIX7 pad 2: Net-(NIX7-µ) -> Net-(NIX1-µ)
- NIX7 pad 3: Net-(NIX7-P) -> Net-(NIX1-P)
- NIX7 pad 4: Net-(NIX7--) -> Net-(NIX1--)
- NIX7 pad 5: Net-(NIX7-+) -> Net-(NIX1-+)
- NIX7 pad 6: Net-(NIX7-m) -> Net-(NIX1-m)
- NIX7 pad 7: Net-(NIX7-M) -> Net-(NIX1-M)
- NIX7 pad 8: Net-(NIX7-k) -> Net-(NIX1-k)
- NIX7 pad 9: Net-(NIX7-П) -> Net-(NIX1-П)
- Q3 pad 2: GND -> +170V
- R1 pad 1: Net-(NE1-A) -> Net-(Q1-C)
- R1 pad 2: +170V -> +12V
- R10 pad 1: Net-(U3-1) -> Net-(Q4-C)
- R10 pad 2: Net-(Q2-B) -> +12V
- R11 pad 1: Net-(U3-2) -> Net-(Q5-C)
- R11 pad 2: Net-(Q3-B) -> +12V
- R12 pad 1: Net-(U3-3) -> Net-(NIX3-~{A})
- R12 pad 2: Net-(Q4-B) -> Net-(Q3-C)
- R13 pad 1: Net-(Q1-C) -> Net-(Q3-B)
- R13 pad 2: +12V -> Net-(U3-HV31)
- R14 pad 1: Net-(Q2-C) -> Net-(NIX4-~{A})
- R14 pad 2: +12V -> Net-(Q6-C)
- R15 pad 1: Net-(Q3-C) -> Net-(Q6-B)
- R15 pad 2: +12V -> Net-(U3-HV32)
- R16 pad 1: Net-(Q4-C) -> Net-(Q7-B)
- R16 pad 2: +12V -> Net-(U5-HV1)
- R2 pad 1: Net-(NE2-A) -> Net-(NIX1-~{A})
- R2 pad 2: +170V -> Net-(Q3-C)
- R3 pad 1: Net-(NIX5-~{A}) -> Net-(U2-0)
- R3 pad 2: +170V -> Net-(Q1-B)
- R4 pad 1: Net-(NIX6-~{A}) -> Net-(U2-1)
- R4 pad 2: +170V -> Net-(Q2-B)
- R5 pad 1: Net-(NIX7-~{A}) -> Net-(U2-2)
- R5 pad 2: +170V -> Net-(Q4-B)
- R9 pad 1: Net-(U3-0) -> Net-(NIX2-~{A})
- R9 pad 2: Net-(Q1-B) -> Net-(Q3-C)
- U1 pad 1: Net-(NIX6-n) -> +12V
- U1 pad 2: Net-(NIX6-%) -> GND
- U1 pad 3: Net-(NIX6-П) -> +5V
- U3 pad 1: +5V -> Net-(NIX11-M)
- U3 pad 15: unconnected-(U3-8-Pad15) -> Net-(NIX12-P)
- U3 pad 16: unconnected-(U3-7-Pad16) -> Net-(NIX12-µ)
- U3 pad 17: unconnected-(U3-6-Pad17) -> Net-(NIX12--)
- U3 pad 18: unconnected-(U3-5-Pad18) -> Net-(NIX12-m)
- U3 pad 19: unconnected-(U3-4-Pad19) -> Net-(NIX12-%)
- U3 pad 2: GND -> Net-(NIX11-П)
- U3 pad 20: Net-(U3-3) -> Net-(NIX12-k)
- U3 pad 21: Net-(U3-2) -> Net-(U3-HV31)
- U3 pad 22: Net-(U3-1) -> Net-(U3-HV32)
- U3 pad 23: Net-(U3-0) -> Net-(U3-DATAOUT)
- U3 pad 3: unconnected-(U3-+3V3-Pad3) -> Net-(NIX11-n)
- U3 pad 4: unconnected-(U3-29-Pad4) -> Net-(NIX11-+)
- U3 pad 5: unconnected-(U3-28-Pad5) -> Net-(NIX11-P)
- U3 pad 6: unconnected-(U3-27-Pad6) -> Net-(NIX11-µ)
- U3 pad 7: unconnected-(U3-26-Pad7) -> Net-(NIX11--)
- U3 pad 8: unconnected-(U3-15-Pad8) -> Net-(NIX11-m)
- U3 pad 9: unconnected-(U3-14-Pad9) -> Net-(NIX11-%)
- U5 pad 1: +12V -> Net-(NE8-K)
- U5 pad 2: GND -> Net-(NE9-K)
- U5 pad 3: +5V -> Net-(NE10-K)
Routing:
- net Net-(NE8-K): track 0.00 -> 226.5 mm, vias 0 -> 1
- net Net-(NE17-K): track 0.00 -> 226.0 mm, vias 0 -> 1
- net Net-(NE9-K): track 0.00 -> 225.9 mm, vias 0 -> 1
- net Net-(NE16-K): track 0.00 -> 225.4 mm, vias 0 -> 1
- net Net-(NE10-K): track 0.00 -> 225.2 mm, vias 0 -> 1
- net Net-(NE15-K): track 0.00 -> 224.7 mm, vias 0 -> 1
- net Net-(NE11-K): track 0.00 -> 224.5 mm, vias 0 -> 1
- net Net-(NE14-K): track 0.00 -> 224.0 mm, vias 0 -> 1
- net Net-(NE12-K): track 0.00 -> 223.8 mm, vias 0 -> 1
- net Net-(NE13-K): track 0.00 -> 223.3 mm, vias 0 -> 1
- net Net-(U5-HV1): track 0.00 -> 220.7 mm
- net unconnected-(U5-HV30-Pad20): track 0.00 -> 218.5 mm
- net Net-(U5-HV2): track 0.00 -> 218.2 mm
- net unconnected-(U5-HV29-Pad19): track 0.00 -> 216.0 mm
- net Net-(U5-HV3): track 0.00 -> 215.7 mm
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- removed copper zone on B.Cu, net GND
- removed copper zone on F.Cu, net GND
Other:
- board size 110 x 75 mm -> 236 x 113 mm
- copper layers 2 -> 4
- board text removed: "A totally useless device... A manifestation of the sins of man... A abhorrence upon gods land... UwU"
- board text removed: "Beeg Controlly Boi"
- board text removed: "Beeg Shocky Boi"
- board text removed: "FeriNixie {dblquote}Thing{dblquote} V1 Created with Love by Ferinix"
- board text removed: "OwO Whats This?"
- board text removed: "The {dblquote}Thing{dblquote}"
- board text removed: "UwU"

Commit message: Adjustments
Parts:
- removed the REF** at (218.0, 106.0)
- removed the REF** at (197.0, 137.0)
- removed the REF** at (121.0, 75.0)
- removed the REF** at (239.0, 137.0)
- removed the REF** at (176.0, 75.0)
- removed the REF** at (58.0, 106.0)
- removed the REF** at (37.0, 75.0)
- removed the REF** at (100.0, 106.0)
- removed the REF** at (155.0, 75.0)
- removed the REF** at (197.0, 106.0)
- removed the REF** at (121.0, 137.0)
- removed the REF** at (176.0, 137.0)
- removed the REF** at (155.0, 106.0)
- removed the REF** at (239.0, 106.0)
- removed the REF** at (79.0, 106.0)
- removed the REF** at (37.0, 106.0)
- removed the REF** at (58.0, 75.0)
- removed the REF** at (37.0, 137.0)
- removed the REF** at (239.0, 75.0)
- removed the REF** at (100.0, 75.0)
- removed the REF** at (176.0, 106.0)
- removed the REF** at (197.0, 75.0)
- removed the REF** at (155.0, 137.0)
- removed the REF** at (79.0, 75.0)
- removed the REF** at (218.0, 137.0)
- removed the REF** at (58.0, 137.0)
- removed the REF** at (100.0, 137.0)
- removed the REF** at (79.0, 137.0)
- removed the REF** at (218.0, 75.0)
- removed the REF** at (121.0, 106.0)
- added ?: , , F.Cu at (115.9, 46.9)
- added ?: , , F.Cu at (26.9, 46.9)
- added C7: 100nF, Capacitor_SMD:C_0402_1005Metric, B.Cu at (319.9, 165.9)
- added C8: 100nF, Capacitor_SMD:C_0402_1005Metric, B.Cu at (319.9, 167.9)
- added Q10: MMBTA42, NixFootprints:SOT-23 No Courtyard, B.Cu at (158.0, 131.5)
- added Q100: MMBTA42, NixFootprints:SOT-23 No Courtyard, B.Cu at (334.3, 97.5)
- added Q101: MMBTA42, NixFootprints:SOT-23 No Courtyard, B.Cu at (334.3, 102.0)
- added Q102: MMBTA42, NixFootprints:SOT-23 No Courtyard, B.Cu at (334.3, 106.4)
- added Q103: MMBTA42, NixFootprints:SOT-23 No Courtyard, B.Cu at (334.3, 110.9)
- added Q104: MMBTA42, NixFootprints:SOT-23 No Courtyard, B.Cu at (334.3, 115.3)
- added Q105: MMBTA42, NixFootprints:SOT-23 No Courtyard, B.Cu at (334.3, 119.8)
- added Q106: MMBTA42, NixFootprints:SOT-23 No Courtyard, B.Cu at (334.3, 124.2)
- added Q107: MMBTA42, NixFootprints:SOT-23 No Courtyard, B.Cu at (334.3, 128.7)
- added Q108: MMBTA42, NixFootprints:SOT-23 No Courtyard, B.Cu at (334.3, 133.1)
- added Q109: MMBTA42, NixFootprints:SOT-23 No Courtyard, B.Cu at (334.3, 137.6)
- added Q11: MMBTA42, NixFootprints:SOT-23 No Courtyard, B.Cu at (173.0, 145.5)
- added Q110: MMBTA42, NixFootprints:SOT-23 No Courtyard, B.Cu at (334.3, 142.0)
- added Q111: MMBTA42, NixFootprints:SOT-23 No Courtyard, B.Cu at (334.3, 146.5)
- added Q112: MMBTA42, NixFootprints:SOT-23 No Courtyard, B.Cu at (334.3, 150.9)
- added Q113: MMBTA42, NixFootprints:SOT-23 No Courtyard, B.Cu at (329.4, 93.1)
- added Q114: MMBTA42, NixFootprints:SOT-23 No Courtyard, B.Cu at (329.4, 97.5)
- added Q115: MMBTA42, NixFootprints:SOT-23 No Courtyard, B.Cu at (329.4, 102.0)
- added Q116: MMBTA42, NixFootprints:SOT-23 No Courtyard, B.Cu at (329.4, 106.4)
- added Q117: MMBTA42, NixFootprints:SOT-23 No Courtyard, B.Cu at (329.4, 110.9)
- added Q118: MMBTA42, NixFootprints:SOT-23 No Courtyard, B.Cu at (329.4, 115.3)
- added Q119: MMBTA42, NixFootprints:SOT-23 No Courtyard, B.Cu at (329.4, 119.8)
- added Q12: MMBTA42, NixFootprints:SOT-23 No Courtyard, B.Cu at (179.0, 145.5)
- added Q120: MMBTA42, NixFootprints:SOT-23 No Courtyard, B.Cu at (329.4, 124.2)
- added Q121: MMBTA42, NixFootprints:SOT-23 No Courtyard, B.Cu at (329.4, 128.7)
- added Q122: MMBTA42, NixFootprints:SOT-23 No Courtyard, B.Cu at (329.4, 133.1)
- added Q123: MMBTA42, NixFootprints:SOT-23 No Courtyard, B.Cu at (329.4, 137.6)
- added Q124: MMBTA42, NixFootprints:SOT-23 No Courtyard, B.Cu at (329.4, 142.0)
- added Q125: MMBTA42, NixFootprints:SOT-23 No Courtyard, B.Cu at (329.4, 146.5)
- added Q126: MMBTA42, NixFootprints:SOT-23 No Courtyard, B.Cu at (329.4, 150.9)
- added Q127: MMBTA42, NixFootprints:SOT-23 No Courtyard, B.Cu at (324.5, 93.1)
- added Q128: MMBTA42, NixFootprints:SOT-23 No Courtyard, B.Cu at (324.5, 97.5)
- added Q129: MMBTA42, NixFootprints:SOT-23 No Courtyard, B.Cu at (324.5, 102.0)
- added Q13: MMBTA42, NixFootprints:SOT-23 No Courtyard, B.Cu at (173.0, 142.0)
- added Q130: MMBTA42, NixFootprints:SOT-23 No Courtyard, B.Cu at (324.5, 106.4)
- added Q131: MMBTA42, NixFootprints:SOT-23 No Courtyard, B.Cu at (324.5, 110.9)
- added Q132: MMBTA42, NixFootprints:SOT-23 No Courtyard, B.Cu at (324.5, 115.3)
- added Q133: MMBTA42, NixFootprints:SOT-23 No Courtyard, B.Cu at (324.5, 119.8)
- added Q134: MMBTA42, NixFootprints:SOT-23 No Courtyard, B.Cu at (324.5, 124.2)
- added Q135: MMBTA42, NixFootprints:SOT-23 No Courtyard, B.Cu at (324.5, 128.7)
- added Q136: MMBTA42, NixFootprints:SOT-23 No Courtyard, B.Cu at (324.5, 133.1)
- added Q137: MMBTA42, NixFootprints:SOT-23 No Courtyard, B.Cu at (324.5, 137.6)
- added Q138: MMBTA42, NixFootprints:SOT-23 No Courtyard, B.Cu at (324.5, 142.0)
- added Q139: MMBTA42, NixFootprints:SOT-23 No Courtyard, B.Cu at (324.5, 146.5)
- added Q14: MMBTA42, NixFootprints:SOT-23 No Courtyard, B.Cu at (179.0, 142.0)
- added Q140: MMBTA42, NixFootprints:SOT-23 No Courtyard, B.Cu at (324.5, 150.9)
- added Q141: MMBTA42, NixFootprints:SOT-23 No Courtyard, B.Cu at (319.6, 93.1)
- added Q142: MMBTA42, NixFootprints:SOT-23 No Courtyard, B.Cu at (319.6, 97.5)
- added Q143: MMBTA42, NixFootprints:SOT-23 No Courtyard, B.Cu at (319.6, 102.0)
- added Q144: MMBTA42, NixFootprints:SOT-23 No Courtyard, B.Cu at (319.6, 106.4)
- added Q145: MMBTA42, NixFootprints:SOT-23 No Courtyard, B.Cu at (319.6, 110.9)
- added Q146: MMBTA42, NixFootprints:SOT-23 No Courtyard, B.Cu at (319.6, 115.3)
- added Q147: MMBTA42, NixFootprints:SOT-23 No Courtyard, B.Cu at (319.6, 119.8)
- added Q148: MMBTA42, NixFootprints:SOT-23 No Courtyard, B.Cu at (319.6, 124.2)
- added Q149: MMBTA42, NixFootprints:SOT-23 No Courtyard, B.Cu at (319.6, 128.7)
- added Q15: MMBTA42, NixFootprints:SOT-23 No Courtyard, B.Cu at (173.0, 138.5)
- added Q150: MMBTA42, NixFootprints:SOT-23 No Courtyard, B.Cu at (319.6, 133.1)
- added Q151: MMBTA42, NixFootprints:SOT-23 No Courtyard, F.Cu at (335.5, 218.4)
- added Q152: MMBTA42, NixFootprints:SOT-23 No Courtyard, F.Cu at (335.5, 222.7)
- added Q153: MMBTA42, NixFootprints:SOT-23 No Courtyard, F.Cu at (335.5, 226.9)
- added Q154: MMBTA42, NixFootprints:SOT-23 No Courtyard, F.Cu at (335.5, 231.1)
- added Q155: MMBTA42, NixFootprints:SOT-23 No Courtyard, F.Cu at (335.5, 235.4)
- added Q156: MMBTA42, NixFootprints:SOT-23 No Courtyard, F.Cu at (335.5, 239.6)
- added Q157: MMBTA42, NixFootprints:SOT-23 No Courtyard, F.Cu at (339.8, 218.4)
- added Q158: MMBTA42, NixFootprints:SOT-23 No Courtyard, F.Cu at (339.8, 222.7)
- added Q159: MMBTA42, NixFootprints:SOT-23 No Courtyard, F.Cu at (339.8, 226.9)
- added Q16: MMBTA42, NixFootprints:SOT-23 No Courtyard, B.Cu at (179.0, 138.5)
- added Q160: MMBTA42, NixFootprints:SOT-23 No Courtyard, F.Cu at (339.8, 231.1)
- added Q161: MMBTA42, NixFootprints:SOT-23 No Courtyard, F.Cu at (339.8, 235.4)
- added Q162: MMBTA42, NixFootprints:SOT-23 No Courtyard, F.Cu at (339.8, 239.6)
- added Q163: MMBTA42, NixFootprints:SOT-23 No Courtyard, F.Cu at (344.2, 218.4)
- added Q164: MMBTA42, NixFootprints:SOT-23 No Courtyard, F.Cu at (344.2, 222.7)
- added Q165: MMBTA42, NixFootprints:SOT-23 No Courtyard, F.Cu at (344.2, 226.9)
- added Q166: MMBTA42, NixFootprints:SOT-23 No Courtyard, F.Cu at (344.2, 231.1)
- added Q167: MMBTA42, NixFootprints:SOT-23 No Courtyard, F.Cu at (344.2, 235.4)
- added Q168: MMBTA42, NixFootprints:SOT-23 No Courtyard, F.Cu at (344.2, 239.6)
- added Q17: MMBTA42, NixFootprints:SOT-23 No Courtyard, B.Cu at (173.0, 135.0)
- added Q18: MMBTA42, NixFootprints:SOT-23 No Courtyard, B.Cu at (179.0, 135.0)
- added Q19: MMBTA42, NixFootprints:SOT-23 No Courtyard, B.Cu at (173.0, 131.5)
- added Q20: MMBTA42, NixFootprints:SOT-23 No Courtyard, B.Cu at (179.0, 131.5)
- added Q21: MMBTA42, NixFootprints:SOT-23 No Courtyard, B.Cu at (194.0, 145.5)
- added Q22: MMBTA42, NixFootprints:SOT-23 No Courtyard, B.Cu at (200.0, 145.5)
- added Q23: MMBTA42, NixFootprints:SOT-23 No Courtyard, B.Cu at (194.0, 142.0)
- added Q24: MMBTA42, NixFootprints:SOT-23 No Courtyard, B.Cu at (200.0, 142.0)
- added Q25: MMBTA42, NixFootprints:SOT-23 No Courtyard, B.Cu at (194.0, 138.5)
- added Q26: MMBTA42, NixFootprints:SOT-23 No Courtyard, B.Cu at (200.0, 138.5)
- added Q27: MMBTA42, NixFootprints:SOT-23 No Courtyard, B.Cu at (194.0, 135.0)
- added Q28: MMBTA42, NixFootprints:SOT-23 No Courtyard, B.Cu at (200.0, 135.0)
- added Q29: MMBTA42, NixFootprints:SOT-23 No Courtyard, B.Cu at (194.0, 131.5)
- added Q30: MMBTA42, NixFootprints:SOT-23 No Courtyard, B.Cu at (200.0, 131.5)
- added Q31: MMBTA42, NixFootprints:SOT-23 No Courtyard, B.Cu at (215.0, 145.5)
- added Q32: MMBTA42, NixFootprints:SOT-23 No Courtyard, B.Cu at (221.0, 145.5)
- added Q33: MMBTA42, NixFootprints:SOT-23 No Courtyard, B.Cu at (215.0, 142.0)
- added Q34: MMBTA42, NixFootprints:SOT-23 No Courtyard, B.Cu at (221.0, 142.0)
- added Q35: MMBTA42, NixFootprints:SOT-23 No Courtyard, B.Cu at (215.0, 138.5)
- added Q36: MMBTA42, NixFootprints:SOT-23 No Courtyard, B.Cu at (221.0, 138.5)
- added Q37: MMBTA42, NixFootprints:SOT-23 No Courtyard, B.Cu at (215.0, 135.0)
- added Q38: MMBTA42, NixFootprints:SOT-23 No Courtyard, B.Cu at (221.0, 135.0)
- added Q39: MMBTA42, NixFootprints:SOT-23 No Courtyard, B.Cu at (215.0, 131.5)
- added Q40: MMBTA42, NixFootprints:SOT-23 No Courtyard, B.Cu at (221.0, 131.5)
- added Q41: MMBTA42, NixFootprints:SOT-23 No Courtyard, B.Cu at (236.0, 145.5)
- added Q42: MMBTA42, NixFootprints:SOT-23 No Courtyard, B.Cu at (242.0, 145.5)
- added Q43: MMBTA42, NixFootprints:SOT-23 No Courtyard, B.Cu at (236.0, 142.0)
- added Q44: MMBTA42, NixFootprints:SOT-23 No Courtyard, B.Cu at (242.0, 142.0)
- added Q45: MMBTA42, NixFootprints:SOT-23 No Courtyard, B.Cu at (236.0, 138.5)
- added Q46: MMBTA42, NixFootprints:SOT-23 No Courtyard, B.Cu at (242.0, 138.5)
- added Q47: MMBTA42, NixFootprints:SOT-23 No Courtyard, B.Cu at (236.0, 135.0)
- added Q48: MMBTA42, NixFootprints:SOT-23 No Courtyard, B.Cu at (242.0, 135.0)
- added Q49: MMBTA42, NixFootprints:SOT-23 No Courtyard, B.Cu at (236.0, 131.5)
- added Q50: MMBTA42, NixFootprints:SOT-23 No Courtyard, B.Cu at (242.0, 131.5)
- added Q51: MMBTA42, NixFootprints:SOT-23 No Courtyard, B.Cu at (152.0, 114.5)
- added Q52: MMBTA42, NixFootprints:SOT-23 No Courtyard, B.Cu at (158.0, 114.5)
- added Q53: MMBTA42, NixFootprints:SOT-23 No Courtyard, B.Cu at (152.0, 111.0)
- added Q54: MMBTA42, NixFootprints:SOT-23 No Courtyard, B.Cu at (158.0, 111.0)
- added Q55: MMBTA42, NixFootprints:SOT-23 No Courtyard, B.Cu at (152.0, 107.5)
- added Q56: MMBTA42, NixFootprints:SOT-23 No Courtyard, B.Cu at (158.0, 107.5)
- added Q57: MMBTA42, NixFootprints:SOT-23 No Courtyard, B.Cu at (152.0, 104.0)
- added Q58: MMBTA42, NixFootprints:SOT-23 No Courtyard, B.Cu at (158.0, 104.0)
- added Q59: MMBTA42, NixFootprints:SOT-23 No Courtyard, B.Cu at (152.0, 100.5)
- added Q60: MMBTA42, NixFootprints:SOT-23 No Courtyard, B.Cu at (158.0, 100.5)
- added Q61: MMBTA42, NixFootprints:SOT-23 No Courtyard, B.Cu at (173.0, 114.5)
- added Q62: MMBTA42, NixFootprints:SOT-23 No Courtyard, B.Cu at (179.0, 114.5)
- added Q63: MMBTA42, NixFootprints:SOT-23 No Courtyard, B.Cu at (173.0, 111.0)
- added Q64: MMBTA42, NixFootprints:SOT-23 No Courtyard, B.Cu at (179.0, 111.0)
- added Q65: MMBTA42, NixFootprints:SOT-23 No Courtyard, B.Cu at (173.0, 107.5)
- added Q66: MMBTA42, NixFootprints:SOT-23 No Courtyard, B.Cu at (179.0, 107.5)
- added Q67: MMBTA42, NixFootprints:SOT-23 No Courtyard, B.Cu at (173.0, 104.0)
- added Q68: MMBTA42, NixFootprints:SOT-23 No Courtyard, B.Cu at (179.0, 104.0)
- added Q69: MMBTA42, NixFootprints:SOT-23 No Courtyard, B.Cu at (173.0, 100.5)
- added Q70: MMBTA42, NixFootprints:SOT-23 No Courtyard, B.Cu at (179.0, 100.5)
- added Q71: MMBTA42, NixFootprints:SOT-23 No Courtyard, B.Cu at (344.1, 93.1)
- added Q72: MMBTA42, NixFootprints:SOT-23 No Courtyard, B.Cu at (344.1, 97.5)
- added Q73: MMBTA42, NixFootprints:SOT-23 No Courtyard, B.Cu at (344.1, 102.0)
- added Q74: MMBTA42, NixFootprints:SOT-23 No Courtyard, B.Cu at (344.1, 106.4)
- added Q75: MMBTA42, NixFootprints:SOT-23 No Courtyard, B.Cu at (344.1, 110.9)
- added Q76: MMBTA42, NixFootprints:SOT-23 No Courtyard, B.Cu at (344.1, 115.3)
- added Q77: MMBTA42, NixFootprints:SOT-23 No Courtyard, B.Cu at (344.1, 119.8)
- added Q78: MMBTA42, NixFootprints:SOT-23 No Courtyard, B.Cu at (344.1, 124.2)
- added Q79: MMBTA42, NixFootprints:SOT-23 No Courtyard, B.Cu at (344.1, 128.7)
- added Q80: MMBTA42, NixFootprints:SOT-23 No Courtyard, B.Cu at (344.1, 133.1)
- added Q81: MMBTA42, NixFootprints:SOT-23 No Courtyard, B.Cu at (344.1, 137.6)
- added Q82: MMBTA42, NixFootprints:SOT-23 No Courtyard, B.Cu at (344.1, 142.0)
- added Q83: MMBTA42, NixFootprints:SOT-23 No Courtyard, B.Cu at (344.1, 146.5)
- added Q84: MMBTA42, NixFootprints:SOT-23 No Courtyard, B.Cu at (344.1, 150.9)
- added Q85: MMBTA42, NixFootprints:SOT-23 No Courtyard, B.Cu at (339.2, 93.1)
- added Q86: MMBTA42, NixFootprints:SOT-23 No Courtyard, B.Cu at (339.2, 97.5)
- added Q87: MMBTA42, NixFootprints:SOT-23 No Courtyard, B.Cu at (339.2, 102.0)
- added Q88: MMBTA42, NixFootprints:SOT-23 No Courtyard, B.Cu at (339.2, 106.4)
- added Q89: MMBTA42, NixFootprints:SOT-23 No Courtyard, B.Cu at (339.2, 110.9)
- added Q90: MMBTA42, NixFootprints:SOT-23 No Courtyard, B.Cu at (339.2, 115.3)
- added Q91: MMBTA42, NixFootprints:SOT-23 No Courtyard, B.Cu at (339.2, 119.8)
- added Q92: MMBTA42, NixFootprints:SOT-23 No Courtyard, B.Cu at (339.2, 124.2)
- added Q93: MMBTA42, NixFootprints:SOT-23 No Courtyard, B.Cu at (339.2, 128.7)
- added Q94: MMBTA42, NixFootprints:SOT-23 No Courtyard, B.Cu at (339.2, 133.1)
- added Q95: MMBTA42, NixFootprints:SOT-23 No Courtyard, B.Cu at (339.2, 137.6)
- added Q96: MMBTA42, NixFootprints:SOT-23 No Courtyard, B.Cu at (339.2, 142.0)
- added Q97: MMBTA42, NixFootprints:SOT-23 No Courtyard, B.Cu at (339.2, 146.5)
- added Q98: MMBTA42, NixFootprints:SOT-23 No Courtyard, B.Cu at (339.2, 150.9)
- added Q99: MMBTA42, NixFootprints:SOT-23 No Courtyard, B.Cu at (334.3, 93.1)
- added R100: 10K, Resistor_SMD:R_0402_1005Metric, B.Cu at (208.5, 176.4)
- added R101: 10K, Resistor_SMD:R_0402_1005Metric, B.Cu at (208.5, 178.4)
- added R102: 10K, Resistor_SMD:R_0402_1005Metric, B.Cu at (208.5, 180.4)
- added R103: 10K, Resistor_SMD:R_0402_1005Metric, B.Cu at (208.5, 182.4)
- added R104: 10K, Resistor_SMD:R_0402_1005Metric, B.Cu at (208.5, 184.4)
- added R105: 10K, Resistor_SMD:R_0402_1005Metric, B.Cu at (208.5, 186.4)
- added R106: 10K, Resistor_SMD:R_0402_1005Metric, B.Cu at (208.5, 188.4)
- added R107: 10K, Resistor_SMD:R_0402_1005Metric, B.Cu at (205.6, 164.5)
- added R108: 10K, Resistor_SMD:R_0402_1005Metric, B.Cu at (205.6, 166.5)
- added R109: 10K, Resistor_SMD:R_0402_1005Metric, B.Cu at (205.6, 168.5)
- added R110: 10K, Resistor_SMD:R_0402_1005Metric, B.Cu at (205.6, 170.5)
- added R111: 10K, Resistor_SMD:R_0402_1005Metric, B.Cu at (205.6, 172.5)
- added R112: 10K, Resistor_SMD:R_0402_1005Metric, B.Cu at (205.6, 174.4)
- added R113: 10K, Resistor_SMD:R_0402_1005Metric, B.Cu at (205.6, 176.4)
- added R114: 10K, Resistor_SMD:R_0402_1005Metric, B.Cu at (205.6, 178.4)
- added R115: 10K, Resistor_SMD:R_0402_1005Metric, B.Cu at (205.6, 180.4)
- added R116: 10K, Resistor_SMD:R_0402_1005Metric, B.Cu at (205.6, 182.4)
- added R117: 10K, Resistor_SMD:R_0402_1005Metric, B.Cu at (205.6, 184.4)
- added R118: 10K, Resistor_SMD:R_0402_1005Metric, B.Cu at (205.6, 186.4)
- added R119: 10K, Resistor_SMD:R_0402_1005Metric, B.Cu at (205.6, 188.4)
- added R120: 10K, Resistor_SMD:R_0402_1005Metric, B.Cu at (202.7, 164.5)
- added R121: 10K, Resistor_SMD:R_0402_1005Metric, B.Cu at (202.7, 166.5)
- added R122: 10K, Resistor_SMD:R_0402_1005Metric, B.Cu at (202.7, 168.5)
- added R123: 10K, Resistor_SMD:R_0402_1005Metric, B.Cu at (202.7, 170.5)
- added R124: 10K, Resistor_SMD:R_0402_1005Metric, B.Cu at (202.7, 172.5)
- added R125: 10K, Resistor_SMD:R_0402_1005Metric, B.Cu at (202.7, 174.4)
- added R126: 10K, Resistor_SMD:R_0402_1005Metric, B.Cu at (202.7, 176.4)
- added R127: 10K, Resistor_SMD:R_0402_1005Metric, B.Cu at (202.7, 178.4)
- added R128: 10K, Resistor_SMD:R_0402_1005Metric, B.Cu at (202.7, 180.4)
- added R129: 10K, Resistor_SMD:R_0402_1005Metric, B.Cu at (202.7, 182.4)
- added R130: 10K, Resistor_SMD:R_0402_1005Metric, B.Cu at (202.7, 184.4)
- added R131: 10K, Resistor_SMD:R_0402_1005Metric, B.Cu at (202.7, 186.4)
- added R132: 10K, Resistor_SMD:R_0402_1005Metric, B.Cu at (202.7, 188.4)
- added R133: 10K, Resistor_SMD:R_0402_1005Metric, B.Cu at (199.8, 164.5)
- added R134: 10K, Resistor_SMD:R_0402_1005Metric, B.Cu at (199.8, 166.5)
- added R135: 10K, Resistor_SMD:R_0402_1005Metric, B.Cu at (199.8, 168.5)
- added R136: 10K, Resistor_SMD:R_0402_1005Metric, B.Cu at (199.8, 170.5)
- added R137: 10K, Resistor_SMD:R_0402_1005Metric, B.Cu at (199.8, 172.5)
- added R138: 10K, Resistor_SMD:R_0402_1005Metric, B.Cu at (199.8, 174.4)
- added R139: 10K, Resistor_SMD:R_0402_1005Metric, B.Cu at (199.8, 176.4)
- added R140: 10K, Resistor_SMD:R_0402_1005Metric, B.Cu at (199.8, 178.4)
- added R141: 10K, Resistor_SMD:R_0402_1005Metric, B.Cu at (199.8, 180.4)
- added R142: 10K, Resistor_SMD:R_0402_1005Metric, B.Cu at (199.8, 182.4)
- added R143: 10K, Resistor_SMD:R_0402_1005Metric, B.Cu at (199.8, 184.4)
- added R144: 10K, Resistor_SMD:R_0402_1005Metric, B.Cu at (199.8, 186.4)
- added R145: 10K, Resistor_SMD:R_0402_1005Metric, B.Cu at (199.8, 188.4)
- added R146: 10K, Resistor_SMD:R_0402_1005Metric, B.Cu at (196.8, 164.5)
- added R147: 10K, Resistor_SMD:R_0402_1005Metric, B.Cu at (196.8, 166.5)
- added R148: 10K, Resistor_SMD:R_0402_1005Metric, B.Cu at (196.8, 168.5)
- added R149: 10K, Resistor_SMD:R_0402_1005Metric, B.Cu at (196.8, 170.5)
- added R150: 10K, Resistor_SMD:R_0402_1005Metric, B.Cu at (196.8, 172.5)
- added R151: 10K, Resistor_SMD:R_0402_1005Metric, B.Cu at (196.8, 174.4)
- added R152: 10K, Resistor_SMD:R_0402_1005Metric, B.Cu at (196.8, 176.4)
- added R153: 10K, Resistor_SMD:R_0402_1005Metric, B.Cu at (196.8, 178.4)
- added R154: 10K, Resistor_SMD:R_0402_1005Metric, B.Cu at (196.8, 180.4)
- added R155: 10K, Resistor_SMD:R_0402_1005Metric, B.Cu at (196.8, 182.4)
- added R156: 10K, Resistor_SMD:R_0402_1005Metric, B.Cu at (196.8, 184.4)
- added R157: 10K, Resistor_SMD:R_0402_1005Metric, B.Cu at (196.8, 186.4)
- added R158: 10K, Resistor_SMD:R_0402_1005Metric, B.Cu at (196.8, 188.4)
- added R159: 10K, Resistor_SMD:R_0402_1005Metric, B.Cu at (193.9, 164.5)
- added R160: 10K, Resistor_SMD:R_0402_1005Metric, B.Cu at (193.9, 166.5)
- added R161: 10K, Resistor_SMD:R_0402_1005Metric, B.Cu at (193.9, 168.5)
- added R162: 10K, Resistor_SMD:R_0402_1005Metric, B.Cu at (193.9, 170.5)
- added R163: 10K, Resistor_SMD:R_0402_1005Metric, B.Cu at (193.9, 172.5)
- added R164: 10K, Resistor_SMD:R_0402_1005Metric, B.Cu at (193.9, 174.4)
- added R165: 10K, Resistor_SMD:R_0402_1005Metric, B.Cu at (193.9, 176.4)
- added R166: 1K, Resistor_SMD:R_0402_1005Metric, B.Cu at (193.9, 178.4)
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Connections:
- C3 pad 2: +12V -> +170V
- C4 pad 2: +12V -> +170V_2
- C5 pad 2: +170V -> +5V
- C6 pad 2: +12V -> +5V
- NIX10 pad 10: Net-(NIX1-%) -> Net-(NIX10-%)
- NIX10 pad 11: Net-(NIX1-n) -> Net-(NIX10-n)
- NIX10 pad 2: Net-(NIX1-µ) -> Net-(NIX10-µ)
- NIX10 pad 3: Net-(NIX1-P) -> Net-(NIX10-P)
- NIX10 pad 4: Net-(NIX1--) -> Net-(NIX10--)
- NIX10 pad 5: Net-(NIX1-+) -> Net-(NIX10-+)
- NIX10 pad 6: Net-(NIX1-m) -> Net-(NIX10-m)
- NIX10 pad 7: Net-(NIX1-M) -> Net-(NIX10-M)
- NIX10 pad 8: Net-(NIX1-k) -> Net-(NIX10-k)
- NIX10 pad 9: Net-(NIX1-П) -> Net-(NIX10-П)
- NIX13 pad 10: Net-(NIX1-%) -> Net-(NIX13-%)
- NIX13 pad 11: Net-(NIX1-n) -> Net-(NIX13-n)
- NIX13 pad 2: Net-(NIX1-µ) -> Net-(NIX13-µ)
- NIX13 pad 3: Net-(NIX1-P) -> Net-(NIX13-P)
- NIX13 pad 4: Net-(NIX1--) -> Net-(NIX13--)
- NIX13 pad 5: Net-(NIX1-+) -> Net-(NIX13-+)
- NIX13 pad 6: Net-(NIX1-m) -> Net-(NIX13-m)
- NIX13 pad 7: Net-(NIX1-M) -> Net-(NIX13-M)
- NIX13 pad 8: Net-(NIX1-k) -> Net-(NIX13-k)
- NIX13 pad 9: Net-(NIX1-П) -> Net-(NIX13-П)
- NIX14 pad 10: Net-(NIX11-%) -> Net-(NIX14-%)
- NIX14 pad 11: Net-(NIX11-n) -> Net-(NIX14-n)
- NIX14 pad 2: Net-(NIX11-µ) -> Net-(NIX14-µ)
- NIX14 pad 3: Net-(NIX11-P) -> Net-(NIX14-P)
- NIX14 pad 4: Net-(NIX11--) -> Net-(NIX14--)
- NIX14 pad 5: Net-(NIX11-+) -> Net-(NIX14-+)
- NIX14 pad 6: Net-(NIX11-m) -> Net-(NIX14-m)
- NIX14 pad 7: Net-(NIX11-M) -> Net-(NIX14-M)
- NIX14 pad 8: Net-(NIX11-k) -> Net-(NIX14-k)
- NIX14 pad 9: Net-(NIX11-П) -> Net-(NIX14-П)
- NIX15 pad 10: Net-(NIX12-%) -> Net-(NIX15-%)
- NIX15 pad 11: Net-(NIX12-n) -> Net-(NIX15-n)
- NIX15 pad 2: Net-(NIX12-µ) -> Net-(NIX15-µ)
- NIX15 pad 3: Net-(NIX12-P) -> Net-(NIX15-P)
- NIX15 pad 4: Net-(NIX12--) -> Net-(NIX15--)
- NIX15 pad 5: Net-(NIX12-+) -> Net-(NIX15-+)
- NIX15 pad 6: Net-(NIX12-m) -> Net-(NIX15-m)
- NIX15 pad 7: Net-(NIX12-M) -> Net-(NIX15-M)
- NIX15 pad 8: Net-(NIX12-k) -> Net-(NIX15-k)
- NIX15 pad 9: Net-(NIX12-П) -> Net-(NIX15-П)
- NIX2 pad 10: Net-(NIX11-%) -> Net-(NIX2-%)
- NIX2 pad 11: Net-(NIX11-n) -> Net-(NIX2-n)
- NIX2 pad 2: Net-(NIX11-µ) -> Net-(NIX2-µ)
- NIX2 pad 3: Net-(NIX11-P) -> Net-(NIX2-P)
- NIX2 pad 4: Net-(NIX11--) -> Net-(NIX2--)
- NIX2 pad 5: Net-(NIX11-+) -> Net-(NIX2-+)
- NIX2 pad 6: Net-(NIX11-m) -> Net-(NIX2-m)
- NIX2 pad 7: Net-(NIX11-M) -> Net-(NIX2-M)
- NIX2 pad 8: Net-(NIX11-k) -> Net-(NIX2-k)
- NIX2 pad 9: Net-(NIX11-П) -> Net-(NIX2-П)
- NIX3 pad 10: Net-(NIX12-%) -> Net-(NIX3-%)
- NIX3 pad 11: Net-(NIX12-n) -> Net-(NIX3-n)
- NIX3 pad 2: Net-(NIX12-µ) -> Net-(NIX3-µ)
- NIX3 pad 3: Net-(NIX12-P) -> Net-(NIX3-P)
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Routing:
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- added copper zone on B.Cu, net GND
- added copper zone on F.Cu, net GND
- added copper zone on In1.Cu, net GND
- added copper zone on In2.Cu, net GND

Commit message: Adjustments
Parts:
- moved U18 185.9 mm to (155.8, 91.8), turned to 90 degrees
- moved U17 183.9 mm to (166.2, 91.8), turned to 90 degrees
- moved U16 181.8 mm to (176.8, 91.8), turned to 90 degrees
- moved U15 179.8 mm to (187.2, 91.8), turned to 90 degrees
- moved U14 119.8 mm to (197.8, 91.8), turned to -90 degrees
- moved U13 117.8 mm to (208.2, 91.8), turned to -90 degrees
- moved U12 115.8 mm to (218.8, 91.8), turned to 90 degrees
- moved U11 113.8 mm to (229.2, 91.8), turned to 90 degrees
- moved U10 111.8 mm to (239.8, 91.8), turned to 90 degrees
- moved R28 72.0 mm to (170.5, 142.5), turned to -90 degrees
- moved R34 67.5 mm to (170.5, 132.0), turned to -90 degrees
- moved R26 67.4 mm to (170.5, 146.0), turned to -90 degrees
- moved R32 63.1 mm to (170.5, 135.5), turned to -90 degrees
- moved R35 61.6 mm to (181.5, 131.0), turned to 90 degrees
- moved R27 60.7 mm to (181.5, 145.0), turned to 90 degrees
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Routing:
- net Net-(U5-QA): track 0.00 -> 50.3 mm
- net Net-(U2-QH'): track 0.00 -> 41.7 mm
- net Net-(U4-QH'): track 0.00 -> 41.6 mm
- net Net-(U3-QA): track 0.00 -> 39.9 mm
- net Net-(U4-QH): track 0.00 -> 34.9 mm, vias 0 -> 2
- net Net-(U2-QD): track 0.00 -> 34.7 mm, vias 0 -> 2
- net Net-(U3-QC): track 0.00 -> 34.6 mm
- net Net-(U4-QA): track 0.00 -> 33.2 mm, vias 0 -> 2
- net GND: track 3.10 -> 34.8 mm, vias 2 -> 44
- net Net-(U2-QH): track 0.00 -> 31.2 mm, vias 0 -> 2
- net Net-(U5-QG): track 0.00 -> 30.6 mm
- net Net-(U2-QF): track 0.00 -> 30.4 mm, vias 0 -> 2
- net Net-(U3-QB): track 0.00 -> 26.7 mm, vias 0 -> 2
- net Net-(U3-QF): track 0.00 -> 24.6 mm, vias 0 -> 2
- net Net-(U4-QC): track 0.00 -> 24.5 mm, vias 0 -> 2
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
Commit message: Fixing old stuff
Parts:
- removed the ? at (115.9, 46.9)
- removed C1, C3, C4: 1uF, Capacitor_SMD:C_1206_3216Metric
- removed the REF** at (169.5, 57.5)
- removed U21: OKI-78SR-5_1.5-W36H-C, Converter_DCDC:Converter_DCDC_Murata_OKI-78SR_Vertical
- removed U22, U23: NCH8200HV, NixFootprints:NCH8200HV Through-Hole
Routing:
- net +12V: track 111.5 -> 0.00 mm
- net +170V_2: track 224.1 -> 158.0 mm
- net +170V: track 273.3 -> 271.2 mm
