File: Ferinixie Fun Panel.kicad_sch (KiCad schematic)
At the start: 30 parts, among them Q1 MMBT2222A, Q2 MMBT2222A, Q3 MMBT2222A, Q4 MMBT2222A, U1 HV5122_Flat, U3 RP2040-Tiny, U4 NCH8200HV, U5 OKI-78SR-5_1.5-W36H-C

Commit message: Saving before I restart
Parts:
- removed R1, R2: 100K, Resistor_SMD:R_1206_3216Metric, symbol NixMinis:Mini_R
- added C3, C6: 1uF, Capacitor_SMD:C_1206_3216Metric, symbol NixMinis:Mini_C
- added D1: 75V, symbol Device:D_Zener_Filled
- added NE10, NE11, NE12, NE13, NE14, NE15, NE16, NE17, NE18, NE3, NE4, NE5, NE6, NE7, NE8, NE9: INS-1, NixFootprints:INS-1, symbol NixSymbols:INS-1
- added NIX10, NIX11, NIX12, NIX13, NIX14, NIX15, NIX4, NIX5, NIX6, NIX7, NIX8, NIX9: IN-15A, NixFootprints:IN-15A Stepped, symbol NixSymbols:IN-15A
- added Q3, Q6, Q7, Q8, Q9: MMBTA92, Package_TO_SOT_SMD:SOT-23, symbol Transistor_BJT:MMBTA92
- added R13, R15, R16, R17, R18, R19, R20, R21, R22, R23, R26, R27, R28, R29, R30, R31, R32, R33, R34, R35, R37, R38, R39: 100K, Resistor_SMD:R_1206_3216Metric, symbol NixMinis:Mini_R
- added R14, R25, R36, R40, R42, R43, R44, R46, R47, R48, R50, R51: 20K, Resistor_SMD:R_1206_3216Metric, symbol NixMinis:Mini_R
- added R24, R41, R45, R49, R8: 10K, Resistor_SMD:R_1206_3216Metric, symbol NixMinis:Mini_R
- added U5: HV5122_Flat, Package_QFP:PQFP-44_10x10mm_P0.8mm, symbol NixSymbols:HV5408_Flat
- NE1, NE2: now in the parts list
- R3: renamed from R9; value 1K -> 10K
- R4: renamed from R10; value 1K -> 10K
- R5: renamed from R11; value 1K -> 10K
- R6: renamed from R12; value 1K -> 10K
- U3: renamed from U1; symbol NixSymbols:HV5122_Flat -> NixSymbols:HV5408_Flat
- renumbered C6 to C4, C3 to C5, NIX5 to NIX1, NIX6 to NIX2, NIX7 to NIX3, Q3 to Q4, Q4 to Q5, R13 to R1, R15 to R10, R16 to R11, R5 to R12, R3 to R2, R14 to R7, R4 to R9, U5 to U1, U3 to U2
Connections:
- net +12V: now also U3.30 (VDD); no longer U3.31 (VDD)
- net +170V: now also Q3.2 (E), Q6.2 (E), Q7.2 (E), Q8.2 (E), Q9.2 (E), R19.2, R20.2, R21.2, R22.2, R23.2, R24.2, R26.2, R27.2, R28.2, R29.2, R30.2, R31.2, R32.2, R33.2, R34.2, R35.2, R37.2, R38.2, R39.2, R41.2, R45.2, R49.2, R8.2; no longer R12.2, R2.2, R9.2
- net GND: now also U3.28 (GND), C3.1, C6.1; no longer U3.30 (GND)
- net at Q1.3 (C), R1.1: no longer U3.33 (DIN)
- net at NIX1.10 (%): now also U3.43 (HV9), NIX10.10 (%), NIX13.10 (%), NIX4.10 (%), NIX7.10 (%); no longer U3.36 (HV2)
- net at NIX1.11 (n): now also U3.37 (HV3), NIX10.11 (n), NIX13.11 (n), NIX4.11 (n), NIX7.11 (n); no longer U3.35 (HV1)
- net at NIX1.2 (µ): now also U3.40 (HV6), NIX10.2 (µ), NIX13.2 (µ), NIX4.2 (µ), NIX7.2 (µ); no longer U3.44 (HV10)
- net at NIX1.3 (P): now also U3.39 (HV5), NIX10.3 (P), NIX13.3 (P), NIX4.3 (P), NIX7.3 (P); no longer U3.43 (HV9)
- net at NIX1.4 (-): now also U3.41 (HV7), NIX10.4 (-), NIX13.4 (-), NIX4.4 (-), NIX7.4 (-); no longer U3.42 (HV8)
- net at NIX1.5 (+): now also U3.38 (HV4), NIX10.5 (+), NIX13.5 (+), NIX4.5 (+), NIX7.5 (+); no longer U3.41 (HV7)
- net at NIX1.6 (m): now also U3.42 (HV8), NIX10.6 (m), NIX13.6 (m), NIX4.6 (m), NIX7.6 (m); no longer U3.40 (HV6)
- net at NIX1.7 (M): now also U3.35 (HV1), NIX10.7 (M), NIX13.7 (M), NIX4.7 (M), NIX7.7 (M); no longer U3.39 (HV5)
- net at NIX1.8 (k): now also U3.44 (HV10), NIX10.8 (k), NIX13.8 (k), NIX4.8 (k), NIX7.8 (k); no longer U3.38 (HV4)
- net at NIX1.9 (П): now also U3.36 (HV2), NIX10.9 (П), NIX13.9 (П), NIX4.9 (П), NIX7.9 (П); no longer U3.37 (HV3)
- net at NIX3.10 (%): now also U3.19 (HV29), NIX12.10 (%), NIX15.10 (%), NIX6.10 (%), NIX9.10 (%); no longer U3.12 (HV22)
- net at NIX3.11 (n): now also U3.13 (HV23), NIX12.11 (n), NIX15.11 (n), NIX6.11 (n), NIX9.11 (n); no longer U3.11 (HV21)
- net at NIX3.2 (µ): now also U3.16 (HV26), NIX12.2 (µ), NIX15.2 (µ), NIX6.2 (µ), NIX9.2 (µ); no longer U3.20 (HV30)
- net at NIX3.3 (P): now also U3.15 (HV25), NIX12.3 (P), NIX15.3 (P), NIX6.3 (P), NIX9.3 (P); no longer U3.19 (HV29)
- net at NIX3.4 (-): now also U3.17 (HV27), NIX12.4 (-), NIX15.4 (-), NIX6.4 (-), NIX9.4 (-); no longer U3.18 (HV28)
- net at NIX3.5 (+): now also U3.14 (HV24), NIX12.5 (+), NIX15.5 (+), NIX6.5 (+), NIX9.5 (+); no longer U3.17 (HV27)
- net at NIX3.6 (m): now also U3.18 (HV28), NIX12.6 (m), NIX15.6 (m), NIX6.6 (m), NIX9.6 (m); no longer U3.16 (HV26)
- net at NIX3.7 (M): now also U3.11 (HV21), NIX12.7 (M), NIX15.7 (M), NIX6.7 (M), NIX9.7 (M); no longer U3.15 (HV25)
- net at NIX3.8 (k): now also U3.20 (HV30), NIX12.8 (k), NIX15.8 (k), NIX6.8 (k), NIX9.8 (k); no longer U3.14 (HV24)
- net at NIX3.9 (П): now also U3.12 (HV22), NIX12.9 (П), NIX15.9 (П), NIX6.9 (П), NIX9.9 (П); no longer U3.13 (HV23)
- net at U3.1 (HV11): now also NIX2.7 (M), NIX11.7 (M), NIX14.7 (M), NIX5.7 (M), NIX8.7 (M); no longer NIX2.11 (n)
- net at U3.10 (HV20): now also NIX2.8 (k), NIX11.8 (k), NIX14.8 (k), NIX5.8 (k), NIX8.8 (k); no longer NIX2.2 (µ)
- net at U3.2 (HV12): now also NIX2.9 (П), NIX11.9 (П), NIX14.9 (П), NIX5.9 (П), NIX8.9 (П); no longer NIX2.10 (%)
- net at U3.21 (HV31): now also R13.2; no longer NE1.2 (K)
- net at U3.22 (HV32): now also R15.2; no longer NE2.2 (K)
- net at Q5.3 (C), R11.1: no longer U3.28 (EN)
- net at Q4.3 (C), R10.1: no longer U3.29 (CLK)
- net at U3.3 (HV13): now also NIX2.11 (n), NIX11.11 (n), NIX14.11 (n), NIX5.11 (n), NIX8.11 (n); no longer NIX2.9 (П)
- net at Q2.3 (C), R7.1: no longer U3.32 (STR)
- net at U3.4 (HV14): now also NIX2.5 (+), NIX11.5 (+), NIX14.5 (+), NIX5.5 (+), NIX8.5 (+); no longer NIX2.8 (k)
- net at U3.5 (HV15): now also NIX2.3 (P), NIX11.3 (P), NIX14.3 (P), NIX5.3 (P), NIX8.3 (P); no longer NIX2.7 (M)
- net at U3.6 (HV16): now also NIX2.2 (µ), NIX11.2 (µ), NIX14.2 (µ), NIX5.2 (µ), NIX8.2 (µ); no longer NIX2.6 (m)
- net at U3.7 (HV17): now also NIX2.4 (-), NIX11.4 (-), NIX14.4 (-), NIX5.4 (-), NIX8.4 (-); no longer NIX2.5 (+)
- net at U3.8 (HV18): now also NIX2.6 (m), NIX11.6 (m), NIX14.6 (m), NIX5.6 (m), NIX8.6 (m); no longer NIX2.4 (-)
- net at U3.9 (HV19): now also NIX2.10 (%), NIX11.10 (%), NIX14.10 (%), NIX5.10 (%), NIX8.10 (%); no longer NIX2.3 (P)
- net at NE1.1 (A): now also R19.1
- net at NE2.1 (A): now also R20.1
- new net: NIX12.1 (~{A}), R47.1
- new net: Q8.3 (C), R44.2, R46.2, R47.2
- new net: Q3.3 (C), R12.2, R2.2, R9.2
- new net: NE14.1 (A), R34.1
- new net: NE10.1 (A), R30.1
- new net: NIX10.1 (~{A}), R44.1
- new net: NIX9.1 (~{A}), R43.1
- new net: Q7.3 (C), R40.2, R42.2, R43.2
- new net: NE13.1 (A), R33.1
- new net: NE4.1 (A), R22.1
- new net: NE4.2 (K), U5.41 (HV7)
- new net: NIX5.1 (~{A}), R25.1
- new net: Q6.3 (C), R14.2, R25.2, R36.2
- new net: NE8.1 (A), R28.1
- new net: NIX8.1 (~{A}), R42.1
- new net: NE16.1 (A), R37.1
- new net: Q9.1 (B), R18.1, R49.1
- new net: NE14.2 (K), U5.7 (HV17)
- new net: NE2.2 (K), U5.39 (HV5)
- new net: Q6.1 (B), R15.1, R24.1
- new net: NIX11.1 (~{A}), R46.1
- new net: NE6.1 (A), R26.1
- new net: NIX4.1 (~{A}), R14.1
- new net: NE8.2 (K), U5.1 (HV11)
- new net: NE17.2 (K), U5.10 (HV20)
- new net: NE18.2 (K), U5.11 (HV21)
- new net: NE9.2 (K), U5.2 (HV12)
- new net: NE10.2 (K), U5.3 (HV13)
- new net: R16.2, U5.35 (HV1)
- new net: R17.2, U5.36 (HV2)
- new net: R18.2, U5.37 (HV3)
- new net: NE1.2 (K), U5.38 (HV4)
- new net: NE11.2 (K), U5.4 (HV14)
- new net: NE3.2 (K), U5.40 (HV6)
- new net: NE5.2 (K), U5.42 (HV8)
- new net: NE6.2 (K), U5.43 (HV9)
- new net: NE7.2 (K), U5.44 (HV10)
- new net: NE12.2 (K), U5.5 (HV15)
- new net: NE13.2 (K), U5.6 (HV16)
- new net: NE15.2 (K), U5.8 (HV18)
- new net: NE16.2 (K), U5.9 (HV19)
- new net: NE11.1 (A), R31.1
- new net: NE5.1 (A), R23.1
- new net: Q3.1 (B), R13.1, R8.1
- new net: NE7.1 (A), R27.1
- new net: Q7.1 (B), R16.1, R41.1
- new net: NE18.1 (A), R39.1
- new net: NE3.1 (A), R21.1
- new net: NE17.1 (A), R38.1
- new net: NIX13.1 (~{A}), R48.1
- new net: NE15.1 (A), R35.1
- new net: NE9.1 (A), R29.1
- new net: Q9.3 (C), R48.2, R50.2, R51.2
- new net: NIX6.1 (~{A}), R36.1
- new net: Q8.1 (B), R17.1, R45.1
- new net: NIX7.1 (~{A}), R40.1
- new net: NIX14.1 (~{A}), R50.1
- new net: NE12.1 (A), R32.1
- new net: NIX15.1 (~{A}), R51.1
- no-connect marks 0 -> 28
Other:
- moved on the sheet: U1, U2, U4

Commit message: Adjustments
Parts:
- removed C3: 1uF, Capacitor_SMD:C_1206_3216Metric, symbol NixMinis:Mini_C
- removed D1: 75V, symbol Device:D_Zener_Filled
- removed Q1, Q2, Q4, Q5: MMBT2222A, Package_TO_SOT_SMD:SOT-23, symbol Transistor_BJT:MMBT2222A
- removed Q3, Q6, Q7, Q8, Q9: MMBTA92, Package_TO_SOT_SMD:SOT-23, symbol Transistor_BJT:MMBTA92
- removed R1: 10K, Resistor_SMD:R_1206_3216Metric, symbol NixMinis:Mini_R
- removed U3, U5: HV5122_Flat, Package_QFP:PQFP-44_10x10mm_P0.8mm, symbol NixSymbols:HV5408_Flat
- added C5, C7, C8: 100nF, Capacitor_SMD:C_0402_1005Metric, symbol NixMinis:Mini_C
- added Q1, Q10, Q100, Q101, Q102, Q103, Q104, Q105, Q106, Q107, Q108, Q109, Q11, Q110, Q111, Q112, Q113, Q114, Q115, Q116, Q117, Q118, Q119, Q12, Q120, Q121, Q122, Q123, Q124, Q125, Q126, Q127, Q128, Q129, Q13, Q130, Q131, Q132, Q133, Q134, Q135, Q136, Q137, Q138, Q139, Q14, Q140, Q141, Q142, Q143, Q144, Q145, Q146, Q147, Q148, Q149, Q15, Q150, Q151, Q152, Q153, Q154, Q155, Q156, Q157, Q158, Q159, Q16, Q160, Q161, Q162, Q163, Q164, Q165, Q166, Q167, Q168, Q17, Q18, Q19, Q2, Q20, Q21, Q22, Q23, Q24, Q25, Q26, Q27, Q28, Q29, Q3, Q30, Q31, Q32, Q33, Q34, Q35, Q36, Q37, Q38, Q39, Q4, Q40, Q41, Q42, Q43, Q44, Q45, Q46, Q47, Q48, Q49, Q5, Q50, Q51, Q52, Q53, Q54, Q55, Q56, Q57, Q58, Q59, Q6, Q60, Q61, Q62, Q63, Q64, Q65, Q66, Q67, Q68, Q69, Q7, Q70, Q71, Q72, Q73, Q74, Q75, Q76, Q77, Q78, Q79, Q8, Q80, Q81, Q82, Q83, Q84, Q85, Q86, Q87, Q88, Q89, Q9, Q90, Q91, Q92, Q93, Q94, Q95, Q96, Q97, Q98, Q99: MMBTA42, NixFootprints:SOT-23 No Courtyard, symbol NixMinis:Mini_BJT_NPN
- added R100, R101, R102, R103, R104, R105, R106, R107, R108, R109, R110, R111, R112, R113, R114, R115, R116, R117, R118, R119, R120, R121, R122, R123, R124, R125, R126, R127, R128, R129, R130, R131, R132, R133, R134, R135, R136, R137, R138, R139, R140, R141, R142, R143, R144, R145, R146, R147, R148, R149, R150, R151, R152, R153, R154, R155, R156, R157, R158, R159, R160, R161, R162, R163, R164, R165, R171, R172, R173, R174, R175, R176, R177, R178, R179, R180, R181, R182, R183, R184, R185, R186, R187, R188, R52, R53, R54, R55, R56, R57, R58, R59, R60, R61, R62, R63, R64, R65, R66, R67, R68, R69, R70, R71, R72, R73, R74, R75, R76, R77, R78, R79, R80, R81, R82, R83, R84, R85, R86, R87, R88, R89, R90, R91, R92, R93, R94, R95, R96, R97, R98, R99: 10K, Resistor_SMD:R_0402_1005Metric, symbol NixMinis:Mini_R
- added R12: 20K, Resistor_SMD:R_1206_3216Metric, symbol NixMinis:Mini_R
- added R166, R167, R168, R169, R170: 1K, Resistor_SMD:R_0402_1005Metric, symbol NixMinis:Mini_R
- added R189, R190, R191, R192, R193, R194, R195, R196, R197, R198, R199, R200, R201, R202, R203, R204, R205, R206: 100K, Resistor_SMD:R_1206_3216Metric, symbol NixMinis:Mini_R
- added U1, U10, U11, U12, U13, U14, U15, U16, U17, U18, U19, U2, U3, U39, U4, U40, U5, U6, U7, U8, U9: 74HC595_Slim, Package_SO:SOIC-16_3.9x9.9mm_P1.27mm, symbol NixSymbols:74HC595_Slim
- added U23: NCH8200HV, NixFootprints:NCH8200HV Through-Hole, symbol NixSymbols:NCH8200HV
- added U24, U25, U26, U27, U28, U29, U30, U31, U32, U33, U34, U35, U36, U37, U38: (no value), NixFootprints:PinHeader_1x10_P1.00mm_Vertical, symbol NixSymbols:Pinheader_10
- C6: value 1uF -> 100nF; footprint Capacitor_SMD:C_1206_3216Metric -> Capacitor_SMD:C_0402_1005Metric
- R10, R11, R3, R4, R5, R6, R7, R8: value 10K -> 20K
- R13, R15: value 100K -> 20K
- R16, R17, R18, R19, R20, R21, R22, R23, R26, R27, R28, R29, R30, R31, R32, R33, R34, R35, R37, R38, R39: value 100K -> 10K; footprint Resistor_SMD:R_1206_3216Metric -> Resistor_SMD:R_0402_1005Metric
- R24, R41, R45, R49: footprint Resistor_SMD:R_1206_3216Metric -> Resistor_SMD:R_0402_1005Metric
- R25, R36, R40, R42, R43, R44, R46, R47, R48, R50, R51: value 20K -> 10K; footprint Resistor_SMD:R_1206_3216Metric -> Resistor_SMD:R_0402_1005Metric
- renumbered C5 to C3, R2 to R1, R12 to R2, U2 to U20, U1 to U21, U4 to U22
Connections:
- net +12V: now also U23.1 (12V); no longer C4.2, R10.2, R11.2, R7.2
- net +170V: now also R1.2, R2.2, R3.2, R4.2, R5.2, R6.2, R7.2, R9.2; no longer R19.2, R20.2, R21.2, R22.2, R23.2, R24.2, R26.2, R27.2, R28.2, R29.2, R30.2, R31.2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
- net +5V: now also C6.2, C5.2, C7.2, C8.2, U1.16 (VCC), U10.16 (VCC), U16.16 (VCC), U17.16 (VCC), U18.16 (VCC), U19.16 (VCC), U2.16 (VCC), U3.16 (VCC)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
- net GND: now also C5.1, C7.1, C8.1, Q1.2 (E), Q10.2 (E), Q100.2 (E), Q101.2 (E), Q102.2 (E), Q103.2 (E), Q104.2 (E), Q105.2 (E), Q106.2 (E)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
- net at R47.1: now also U4.7 (QH); no longer NIX12.1 (~{A})
- net at NE14.1 (A): now also R202.1; no longer R34.1
- net at R30.1: now also U2.6 (QG); no longer NE10.1 (A)
- net at NIX10.1 (~{A}): now also R10.1; no longer R44.1
- net at R20.1: now also U1.4 (QE); no longer NE2.1 (A)
- net at U20.22 (1): now also R167.1; no longer R4.1
- net at R43.1: now also U4.3 (QD); no longer NIX9.1 (~{A})
- net at NE13.1 (A): now also R201.1; no longer R33.1
- net at R2.1: now also NIX2.1 (~{A}); no longer NIX3.1 (~{A})
- net at R22.1: now also U1.6 (QG); no longer NE4.1 (A)
- net at NE4.2 (K): now also Q154.3 (C)
- net at NIX5.1 (~{A}): now also R5.1; no longer R25.1
- net at NE8.1 (A): now also R196.1; no longer R28.1
- net at U20.19 (4): now also R170.1
- net at U20.20 (3): now also R169.1; no longer R6.1
- net at U20.21 (2): now also R168.1; no longer R5.1
- net at U20.23 (0): now also R166.1; no longer R3.1
- net at R42.1: now also U4.2 (QC); no longer NIX8.1 (~{A})
- net at NE16.1 (A): now also R204.1; no longer R37.1
- net at R18.1: now also U1.2 (QC); no longer R49.1
- net +170V_2: now reaches R13.2
- net +170V_2: now also C4.2, R10.2, R11.2, R14.2, R15.2, R12.2, R189.2, R190.2, R191.2, R192.2, R193.2, R194.2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
- net at NE14.2 (K): now also Q164.3 (C)
- net at NE2.2 (K): now also Q152.3 (C)
- net at R24.1: now also U2.15 (QA); no longer R15.1
- net at R46.1: now also U4.6 (QG); no longer NIX11.1 (~{A})
- net at R11.1: now also NIX11.1 (~{A})
- net at NE6.1 (A): now also R194.1; no longer R26.1
- net at NIX4.1 (~{A}): now also R4.1; no longer R14.1
- net at NE8.2 (K): now also Q158.3 (C)
- net at NE17.2 (K): now also Q167.3 (C)
- net at NE18.2 (K): now also Q168.3 (C)
- net at NE9.2 (K): now also Q159.3 (C)
- net at NE10.2 (K): now also Q160.3 (C)
- net at R16.2: now also Q1.1 (B)
- net at R17.2: now also Q2.1 (B)
- net at R18.2: now also Q3.1 (B)
- net at NE1.2 (K): now also Q151.3 (C)
- net at NE11.2 (K): now also Q161.3 (C)
- net at NE3.2 (K): now also Q153.3 (C)
- net at NE5.2 (K): now also Q155.3 (C)
- net at NE6.2 (K): now also Q156.3 (C)
- net at NE7.2 (K): now also Q157.3 (C)
- net at NE12.2 (K): now also Q162.3 (C)
- net at NE13.2 (K): now also Q163.3 (C)
- net at NE15.2 (K): now also Q165.3 (C)
- net at NE16.2 (K): now also Q166.3 (C)
- net at R31.1: now also U2.7 (QH); no longer NE11.1 (A)
- net at NE5.1 (A): now also R193.1; no longer R23.1
- net at R8.1: now also NIX8.1 (~{A}); no longer R13.1
- net at R27.1: now also U2.3 (QD); no longer NE7.1 (A)
- net at R41.1: now also U4.1 (QB); no longer R16.1
- net at NE18.1 (A): now also R206.1; no longer R39.1
- net at NE3.1 (A): now also R191.1; no longer R21.1
- net at NE17.1 (A): now also R205.1; no longer R38.1
- net at R48.1: now also U5.15 (QA); no longer NIX13.1 (~{A})
- net at NE1.1 (A): now also R189.1; no longer R19.1
- net at NE15.1 (A): now also R203.1; no longer R35.1
- new net: Q123.1 (B), R138.2
- new net: NIX13.4 (-), Q123.3 (C), U36.3
- new net: R169.2, U1.12 (RCLK), U10.12 (RCLK), U11.12 (RCLK), U12.12 (RCLK), U13.12 (RCLK), U14.12 (RCLK), U15.12 (RCLK), U16.12 (RCLK), U17.12 (RCLK), U18.12 (RCLK), U19.12 (RCLK)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
- new net: Q33.1 (B), R48.2
- new net: Q96.1 (B), R111.2
- new net: NIX10.11 (n), Q96.3 (C), U33.6
- new net: R141.1, U16.5 (QF)
- new net: Q126.1 (B), R141.2
- new net: Q8.1 (B), R23.2
- new net: NIX1.9 (П), Q8.3 (C), U24.8
- new net: Q103.1 (B), R118.2
- new net: NIX11.4 (-), Q103.3 (C), U34.3
- new net: R174.1, U39.1 (QB)
- new net: Q154.1 (B), R174.2
- new net: R90.1, U10.2 (QC)
- new net: Q75.1 (B), R90.2
- new net: Q62.1 (B), R77.2
- new net: NIX7.3 (P), Q62.3 (C), U30.2
- new net: R64.1, U7.15 (QA)
- new net: Q49.1 (B), R64.2
- new net: NIX5.2 (µ), Q41.3 (C), U28.1
- new net: NIX5.7 (M), Q50.3 (C), U28.10
- new net: NIX5.3 (P), Q42.3 (C), U28.2
- new net: NIX5.4 (-), Q43.3 (C), U28.3
- new net: NIX5.5 (+), Q44.3 (C), U28.4
- new net: NIX5.6 (m), Q45.3 (C), U28.5
- new net: NIX5.11 (n), Q46.3 (C), U28.6
- new net: NIX5.10 (%), Q47.3 (C), U28.7
- new net: NIX5.9 (П), Q48.3 (C), U28.8
- new net: NIX5.8 (k), Q49.3 (C), U28.9
- new net: Q42.1 (B), R57.2
- new net: Q32.1 (B), R47.2
- new net: Q74.1 (B), R89.2
- new net: NIX8.5 (+), Q74.3 (C), U31.4
- new net: NIX10.2 (µ), Q91.3 (C), U33.1
- new net: NIX10.7 (M), Q100.3 (C), U33.10
- new net: NIX10.3 (P), Q92.3 (C), U33.2
- new net: NIX10.4 (-), Q93.3 (C), U33.3
- new net: NIX10.5 (+), Q94.3 (C), U33.4
- new net: NIX10.6 (m), Q95.3 (C), U33.5
- new net: NIX10.10 (%), Q97.3 (C), U33.7
- new net: NIX10.9 (П), Q98.3 (C), U33.8
- new net: NIX10.8 (k), Q99.3 (C), U33.9
- new net: R69.1, U7.5 (QF)
- new net: Q54.1 (B), R69.2
- new net: NIX13.2 (µ), Q121.3 (C), U36.1
- new net: NIX13.7 (M), Q130.3 (C), U36.10
- new net: NIX13.3 (P), Q122.3 (C), U36.2
- new net: NIX13.5 (+), Q124.3 (C), U36.4
- new net: NIX13.6 (m), Q125.3 (C), U36.5
- new net: NIX13.11 (n), Q126.3 (C), U36.6
- new net: NIX13.10 (%), Q127.3 (C), U36.7
- new net: NIX13.9 (П), Q128.3 (C), U36.8
- new net: NIX13.8 (k), Q129.3 (C), U36.9
- new net: Q143.1 (B), R158.2
- new net: NIX15.4 (-), Q143.3 (C), U38.3
- new net: Q16.1 (B), R31.2
- new net: NIX2.11 (n), Q16.3 (C), U25.6
- new net: Q31.1 (B), R46.2
- new net: NIX4.2 (µ), Q31.3 (C), U27.1
- new net: NIX4.7 (M), Q40.3 (C), U27.10
- new net: NIX4.3 (P), Q32.3 (C), U27.2
- new net: NIX4.4 (-), Q33.3 (C), U27.3
- new net: NIX4.5 (+), Q34.3 (C), U27.4
- new net: NIX4.6 (m), Q35.3 (C), U27.5
- new net: NIX4.11 (n), Q36.3 (C), U27.6
- new net: NIX4.10 (%), Q37.3 (C), U27.7
- new net: NIX4.9 (П), Q38.3 (C), U27.8
- new net: NIX4.8 (k), Q39.3 (C), U27.9
- new net: R71.1, U7.7 (QH)
- new net: Q56.1 (B), R71.2
- new net: Q104.1 (B), R119.2
- new net: NIX11.5 (+), Q104.3 (C), U34.4
- new net: Q89.1 (B), R104.2
- new net: NIX9.8 (k), Q89.3 (C), U32.9
- new net: R147.1, U17.3 (QD)
- new net: Q132.1 (B), R147.2
- new net: R175.1, U39.2 (QC)
- new net: Q155.1 (B), R175.2
- new net: Q5.1 (B), R20.2
- new net: Q86.1 (B), R101.2
- new net: NIX9.11 (n), Q86.3 (C), U32.6
- new net: Q66.1 (B), R81.2
- new net: NIX7.11 (n), Q66.3 (C), U30.6
- new net: Q77.1 (B), R92.2
- new net: NIX8.10 (%), Q77.3 (C), U31.7
- new net: Q90.1 (B), R105.2
- new net: NIX9.7 (M), Q90.3 (C), U32.10
- new net: Q59.1 (B), R74.2
- new net: NIX6.8 (k), Q59.3 (C), U29.9
- new net: Q7.1 (B), R22.2
- new net: NE2.1 (A), R190.1
- new net: Q158.1 (B), R178.2
- new net: R106.1, U12.2 (QC)
- new net: Q91.1 (B), R106.2
- new net: R179.1, U39.6 (QG)
- new net: Q159.1 (B), R179.2
- new net: R98.1, U11.2 (QC)
- new net: Q83.1 (B), R98.2
- new net: R143.1, U16.7 (QH)
- new net: Q128.1 (B), R143.2
- new net: R81.1, U9.1 (QB)
- new net: R149.1, U17.5 (QF)
- new net: Q134.1 (B), R149.2
- new net: R126.1, U14.6 (QG)
- new net: Q111.1 (B), R126.2
- new net: R146.1, U17.2 (QC)
- new net: Q131.1 (B), R146.2
- new net: R168.2, U1.10 (~{SRCLR}), U10.10 (~{SRCLR}), U11.10 (~{SRCLR}), U12.10 (~{SRCLR}), U13.10 (~{SRCLR}), U14.10 (~{SRCLR}), U15.10 (~{SRCLR}), U16.10 (~{SRCLR}), U17.10 (~{SRCLR}), U18.10 (~{SRCLR}), U19.10 (~{SRCLR})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
- new net: R167.2, U1.11 (SRCLK), U10.11 (SRCLK), U11.11 (SRCLK), U12.11 (SRCLK), U13.11 (SRCLK), U14.11 (SRCLK), U15.11 (SRCLK), U16.11 (SRCLK), U17.11 (SRCLK), U18.11 (SRCLK), U19.11 (SRCLK)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
- new net: R170.2, U1.13 (~{OE}), U10.13 (~{OE}), U11.13 (~{OE}), U12.13 (~{OE}), U13.13 (~{OE}), U14.13 (~{OE}), U15.13 (~{OE}), U16.13 (~{OE}), U17.13 (~{OE}), U18.13 (~{OE}), U19.13 (~{OE})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
- new net: U3.9 (QH'), U4.14 (SER)
- new net: R44.1, U4.4 (QE)
- new net: U4.9 (QH'), U5.14 (SER)
- new net: Q147.1 (B), R162.2
- new net: NIX15.10 (%), Q147.3 (C), U38.7
- new net: R58.1, U6.2 (QC)
- new net: Q43.1 (B), R58.2
- new net: Q136.1 (B), R151.2
- new net: NIX14.11 (n), Q136.3 (C), U37.6
- new net: Q25.1 (B), R40.2
- new net: NIX3.6 (m), Q25.3 (C), U26.5
- new net: R153.1, U18.1 (QB)
- new net: U17.9 (QH'), U18.14 (SER)
- new net: R152.1, U18.15 (QA)
- new net: R154.1, U18.2 (QC)
- new net: R155.1, U18.3 (QD)
- new net: R156.1, U18.4 (QE)
- new net: R157.1, U18.5 (QF)
- new net: R158.1, U18.6 (QG)
- new net: R159.1, U18.7 (QH)
- new net: U18.9 (QH'), U19.14 (SER)
- new net: R80.1, U9.15 (QA)
- new net: Q65.1 (B), R80.2
- new net: Q148.1 (B), R163.2
- new net: NIX15.9 (П), Q148.3 (C), U38.8
- new net: Q164.1 (B), R184.2
- new net: R112.1, U13.15 (QA)
- new net: Q97.1 (B), R112.2
- new net: Q37.1 (B), R52.2
- new net: R17.1, U1.1 (QB)
- new net: NIX6.2 (µ), Q51.3 (C), U29.1
- new net: NIX6.7 (M), Q60.3 (C), U29.10
- new net: NIX6.3 (P), Q52.3 (C), U29.2
- new net: NIX6.4 (-), Q53.3 (C), U29.3
- new net: NIX6.5 (+), Q54.3 (C), U29.4
- new net: NIX6.6 (m), Q55.3 (C), U29.5
- new net: NIX6.11 (n), Q56.3 (C), U29.6
- new net: NIX6.10 (%), Q57.3 (C), U29.7
- new net: NIX6.9 (П), Q58.3 (C), U29.8
- new net: Q138.1 (B), R153.2
- new net: NIX1.10 (%), Q7.3 (C), U24.7
- new net: NIX1.11 (n), Q6.3 (C), U24.6
- new net: NIX1.2 (µ), Q1.3 (C), U24.1
- new net: NIX1.3 (P), Q2.3 (C), U24.2
- new net: NIX1.4 (-), Q3.3 (C), U24.3
- new net: NIX1.5 (+), Q4.3 (C), U24.4
- new net: NIX1.6 (m), Q5.3 (C), U24.5
- new net: NIX1.7 (M), Q10.3 (C), U24.10
- new net: NIX1.8 (k), Q9.3 (C), U24.9
- new net: Q78.1 (B), R93.2
- new net: NIX8.9 (П), Q78.3 (C), U31.8
- new net: Q137.1 (B), R152.2
- new net: NIX14.10 (%), Q137.3 (C), U37.7
- new net: Q27.1 (B), R42.2
- new net: NIX3.10 (%), Q27.3 (C), U26.7
- new net: Q161.1 (B), R181.2
- new net: NIX3.1 (~{A}), R3.1
- new net: NIX3.11 (n), Q26.3 (C), U26.6
- new net: NIX3.2 (µ), Q21.3 (C), U26.1
- new net: NIX3.3 (P), Q22.3 (C), U26.2
- new net: NIX3.4 (-), Q23.3 (C), U26.3
- new net: NIX3.5 (+), Q24.3 (C), U26.4
- new net: NIX3.7 (M), Q30.3 (C), U26.10
- new net: NIX3.8 (k), Q29.3 (C), U26.9
- new net: NIX3.9 (П), Q28.3 (C), U26.8
- new net: Q35.1 (B), R50.2
- new net: Q81.1 (B), R96.2
- new net: NIX9.2 (µ), Q81.3 (C), U32.1
- new net: R99.1, U11.3 (QD)
- new net: Q84.1 (B), R99.2
- new net: R97.1, U11.1 (QB)
- new net: U10.9 (QH'), U11.14 (SER)
- new net: R96.1, U11.15 (QA)
- new net: U11.16 (VCC), U12.16 (VCC), U13.16 (VCC), U15.16 (VCC)
- new net: R100.1, U11.4 (QE)
- new net: R101.1, U11.5 (QF)
- new net: R102.1, U11.6 (QG)
- new net: R103.1, U11.7 (QH)
- new net: U11.9 (QH'), U12.14 (SER)
- new net: NIX9.10 (%), Q87.3 (C), U32.7
- new net: NIX9.3 (P), Q82.3 (C), U32.2
- new net: NIX9.4 (-), Q83.3 (C), U32.3
- new net: NIX9.5 (+), Q84.3 (C), U32.4
- new net: NIX9.6 (m), Q85.3 (C), U32.5
- new net: NIX9.9 (П), Q88.3 (C), U32.8
- new net: R171.1, U19.6 (QG)
- new net: Q151.1 (B), R171.2
- new net: Q69.1 (B), R84.2
- new net: NIX7.8 (k), Q69.3 (C), U30.9
- new net: Q152.1 (B), R172.2
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
Commit message: Fixing old stuff
Parts:
- removed C3, C4: 1uF, Capacitor_SMD:C_1206_3216Metric, symbol NixMinis:Mini_C
- removed U21: OKI-78SR-5_1.5-W36H-C, Converter_DCDC:Converter_DCDC_Murata_OKI-78SR_Vertical, symbol Converter_DCDC:OKI-78SR-5_1.5-W36H-C
- removed U22, U23: NCH8200HV, NixFootprints:NCH8200HV Through-Hole, symbol NixSymbols:NCH8200HV
- added D1: MB6S, Package_TO_SOT_SMD:TO-269AA, symbol Diode_Bridge:MB6S
- added PS1: IRM-05-5, Converter_ACDC:Converter_ACDC_MeanWell_IRM-05-xx_THT, symbol Converter_ACDC:IRM-05-5
- added U21: (no value), Package_SO:JEITA_SOIC-16_3.9x9.9mm_P1.27mm, symbol NixSymbols:CMT8260N0
- C1, C2: footprint Capacitor_SMD:C_1206_3216Metric -> Capacitor_THT:C_Radial_D5.0mm_H5.0mm_P2.00mm
Connections:
- net +12V is gone; now on net +5V: C1.2
- net +170V_2 is gone; now on net +170V: R10.2, R11.2, R12.2, R13.2, R14.2, R15.2, R189.2, R190.2, R191.2, R192.2, R193.2, R194.2, R195.2, R196.2, R197.2, R198.2, R199.2, R200.2, R201.2, R202.2, R203.2, R204.2, R205.2, R206.2
- net +170V: now also C2.2, D1.3 (+)
- net +5V: now also PS1.4 (+Vo), U21.16 (VDD2); no longer C2.2
- net GND: now also PS1.3 (-Vo), U21.8 (GND1); no longer C2.1, C5.1, C6.1, C7.1, C8.1, Q1.2 (E), Q10.2 (E), Q100.2 (E), Q101.2 (E), Q102.2 (E), Q103.2 (E), Q104.2 (E), Q105.2 (E), Q106.2 (E), Q107.2 (E), Q108.2 (E), Q109.2 (E), Q11.2 (E), Q110.2 (E), Q111.2 (E), Q112.2 (E), Q113.2 (E), Q114.2 (E), Q115.2 (E), Q116.2 (E), Q117.2 (E), Q118.2 (E), Q119.2 (E), Q12.2 (E), Q120.2 (E), Q121.2 (E), Q122.2 (E), Q123.2 (E), Q124.2 (E), Q125.2 (E), Q126.2 (E), Q127.2 (E), Q128.2 (E), Q129.2 (E), Q13.2 (E), Q130.2 (E), Q131.2 (E), Q132.2 (E), Q133.2 (E), Q134.2 (E), Q135.2 (E), Q136.2 (E), Q137.2 (E), Q138.2 (E), Q139.2 (E), Q14.2 (E), Q140.2 (E), Q141.2 (E), Q142.2 (E), Q143.2 (E), Q144.2 (E), Q145.2 (E), Q146.2 (E), Q147.2 (E), Q148.2 (E), Q149.2 (E), Q15.2 (E), Q150.2 (E), Q151.2 (E), Q152.2 (E), Q153.2 (E), Q154.2 (E), Q155.2 (E), Q156.2 (E), Q157.2 (E), Q158.2 (E), Q159.2 (E), Q16.2 (E), Q160.2 (E), Q161.2 (E), Q162.2 (E), Q163.2 (E), Q164.2 (E), Q165.2 (E), Q166.2 (E), Q167.2 (E), Q168.2 (E), Q17.2 (E), Q18.2 (E), Q19.2 (E), Q2.2 (E), Q20.2 (E), Q21.2 (E), Q22.2 (E), Q23.2 (E), Q24.2 (E), Q25.2 (E), Q26.2 (E), Q27.2 (E), Q28.2 (E), Q29.2 (E), Q3.2 (E), Q30.2 (E), Q31.2 (E), Q32.2 (E), Q33.2 (E), Q34.2 (E), Q35.2 (E), Q36.2 (E), Q37.2 (E), Q38.2 (E), Q39.2 (E), Q4.2 (E), Q40.2 (E), Q41.2 (E), Q42.2 (E), Q43.2 (E), Q44.2 (E), Q45.2 (E), Q46.2 (E), Q47.2 (E), Q48.2 (E), Q49.2 (E), Q5.2 (E), Q50.2 (E), Q51.2 (E), Q52.2 (E), Q53.2 (E), Q54.2 (E), Q55.2 (E), Q56.2 (E), Q57.2 (E), Q58.2 (E), Q59.2 (E), Q6.2 (E), Q60.2 (E), Q61.2 (E), Q62.2 (E), Q63.2 (E), Q64.2 (E), Q65.2 (E), Q66.2 (E), Q67.2 (E), Q68.2 (E), Q69.2 (E), Q7.2 (E), Q70.2 (E), Q71.2 (E), Q72.2 (E), Q73.2 (E), Q74.2 (E), Q75.2 (E), Q76.2 (E), Q77.2 (E), Q78.2 (E), Q79.2 (E), Q8.2 (E), Q80.2 (E), Q81.2 (E), Q82.2 (E), Q83.2 (E), Q84.2 (E), Q85.2 (E), Q86.2 (E), Q87.2 (E), Q88.2 (E), Q89.2 (E), Q9.2 (E), Q90.2 (E), Q91.2 (E), Q92.2 (E), Q93.2 (E), Q94.2 (E), Q95.2 (E), Q96.2 (E), Q97.2 (E), Q98.2 (E), Q99.2 (E), U1.8 (GND), U10.8 (GND), U11.8 (GND), U12.8 (GND), U13.8 (GND), U14.8 (GND), U15.8 (GND), U16.8 (GND), U17.8 (GND), U18.8 (GND), U19.8 (GND), U2.8 (GND), U3.8 (GND), U4.8 (GND), U40.8 (GND), U5.8 (GND), U6.8 (GND), U7.8 (GND), U8.8 (GND), U9.8 (GND)
- net TBGND: now reaches U1.12 (RCLK), U10.12 (RCLK), U11.12 (RCLK), U12.12 (RCLK), U13.12 (RCLK), U14.12 (RCLK), U15.12 (RCLK), U16.12 (RCLK), U17.12 (RCLK), U18.12 (RCLK), U19.12 (RCLK), U2.12 (RCLK), U3.12 (RCLK), U39.12 (RCLK), U4.12 (RCLK), U40.12 (RCLK), U5.12 (RCLK), U6.12 (RCLK), U7.12 (RCLK), U8.12 (RCLK), U9.12 (RCLK)
- net TBGND: now also C2.1, C5.1, C6.1, C7.1, C8.1, Q1.2 (E), Q10.2 (E), Q100.2 (E), Q101.2 (E), Q102.2 (E), Q103.2 (E), Q104.2 (E), Q105.2 (E), Q106.2 (E), Q107.2 (E), Q108.2 (E), Q109.2 (E), Q11.2 (E), Q110.2 (E), Q111.2 (E), Q112.2 (E), Q113.2 (E), Q114.2 (E), Q115.2 (E), Q116.2 (E), Q117.2 (E), Q118.2 (E), Q119.2 (E), Q12.2 (E), Q120.2 (E), Q121.2 (E), Q122.2 (E), Q123.2 (E), Q124.2 (E), Q125.2 (E), Q126.2 (E), Q127.2 (E), Q128.2 (E), Q129.2 (E), Q13.2 (E), Q130.2 (E), Q131.2 (E), Q132.2 (E), Q133.2 (E), Q134.2 (E), Q135.2 (E), Q136.2 (E), Q137.2 (E), Q138.2 (E), Q139.2 (E), Q14.2 (E), Q140.2 (E), Q141.2 (E), Q142.2 (E), Q143.2 (E), Q144.2 (E), Q145.2 (E), Q146.2 (E), Q147.2 (E), Q148.2 (E), Q149.2 (E), Q15.2 (E), Q150.2 (E), Q151.2 (E), Q152.2 (E), Q153.2 (E), Q154.2 (E), Q155.2 (E), Q156.2 (E), Q157.2 (E), Q158.2 (E), Q159.2 (E), Q16.2 (E), Q160.2 (E), Q161.2 (E), Q162.2 (E), Q163.2 (E), Q164.2 (E), Q165.2 (E), Q166.2 (E), Q167.2 (E), Q168.2 (E), Q17.2 (E), Q18.2 (E), Q19.2 (E), Q2.2 (E), Q20.2 (E), Q21.2 (E), Q22.2 (E), Q23.2 (E), Q24.2 (E), Q25.2 (E), Q26.2 (E), Q27.2 (E), Q28.2 (E), Q29.2 (E), Q3.2 (E), Q30.2 (E), Q31.2 (E), Q32.2 (E), Q33.2 (E), Q34.2 (E), Q35.2 (E), Q36.2 (E), Q37.2 (E), Q38.2 (E), Q39.2 (E), Q4.2 (E), Q40.2 (E), Q41.2 (E), Q42.2 (E), Q43.2 (E), Q44.2 (E), Q45.2 (E), Q46.2 (E), Q47.2 (E), Q48.2 (E), Q49.2 (E), Q5.2 (E), Q50.2 (E), Q51.2 (E), Q52.2 (E), Q53.2 (E), Q54.2 (E), Q55.2 (E), Q56.2 (E), Q57.2 (E), Q58.2 (E), Q59.2 (E), Q6.2 (E), Q60.2 (E), Q61.2 (E), Q62.2 (E), Q63.2 (E), Q64.2 (E), Q65.2 (E), Q66.2 (E), Q67.2 (E), Q68.2 (E), Q69.2 (E), Q7.2 (E), Q70.2 (E), Q71.2 (E), Q72.2 (E), Q73.2 (E), Q74.2 (E), Q75.2 (E), Q76.2 (E), Q77.2 (E), Q78.2 (E), Q79.2 (E), Q8.2 (E), Q80.2 (E), Q81.2 (E), Q82.2 (E), Q83.2 (E), Q84.2 (E), Q85.2 (E), Q86.2 (E), Q87.2 (E), Q88.2 (E), Q89.2 (E), Q9.2 (E), Q90.2 (E), Q91.2 (E), Q92.2 (E), Q93.2 (E), Q94.2 (E), Q95.2 (E), Q96.2 (E), Q97.2 (E), Q98.2 (E), Q99.2 (E), U1.10 (~{SRCLR}), U1.11 (SRCLK), U1.13 (~{OE}), U1.8 (GND), U10.10 (~{SRCLR}), U10.11 (SRCLK), U10.13 (~{OE}), U10.8 (GND), U11.10 (~{SRCLR}), U11.11 (SRCLK), U11.13 (~{OE}), U11.8 (GND), U12.10 (~{SRCLR}), U12.11 (SRCLK), U12.13 (~{OE}), U12.8 (GND), U13.10 (~{SRCLR}), U13.11 (SRCLK), U13.13 (~{OE}), U13.8 (GND), U14.10 (~{SRCLR}), U14.11 (SRCLK), U14.13 (~{OE}), U14.8 (GND), U15.10 (~{SRCLR}), U15.11 (SRCLK), U15.13 (~{OE}), U15.8 (GND), U16.10 (~{SRCLR}), U16.11 (SRCLK), U16.13 (~{OE}), U16.8 (GND), U17.10 (~{SRCLR}), U17.11 (SRCLK), U17.13 (~{OE}), U17.8 (GND), U18.10 (~{SRCLR}), U18.11 (SRCLK), U18.13 (~{OE}), U18.8 (GND), U19.10 (~{SRCLR}), U19.11 (SRCLK), U19.13 (~{OE}), U19.8 (GND), U2.10 (~{SRCLR}), U2.11 (SRCLK), U2.13 (~{OE}), U2.8 (GND), U3.10 (~{SRCLR}), U3.11 (SRCLK), U3.13 (~{OE}), U3.8 (GND), U39.10 (~{SRCLR}), U39.11 (SRCLK), U39.13 (~{OE}), U39.8 (GND), U4.10 (~{SRCLR}), U4.11 (SRCLK), U4.13 (~{OE}), U4.8 (GND), U40.10 (~{SRCLR}), U40.11 (SRCLK), U40.13 (~{OE}), U40.8 (GND), U5.10 (~{SRCLR}), U5.11 (SRCLK), U5.13 (~{OE}), U5.8 (GND), U6.10 (~{SRCLR}), U6.11 (SRCLK), U6.13 (~{OE}), U6.8 (GND), U7.10 (~{SRCLR}), U7.11 (SRCLK), U7.13 (~{OE}), U7.8 (GND), U8.10 (~{SRCLR}), U8.11 (SRCLK), U8.13 (~{OE}), U8.8 (GND), U9.10 (~{SRCLR}), U9.11 (SRCLK), U9.13 (~{OE}), U9.8 (GND), D1.4 (-), U21.11 (OUTE), U21.12 (OUTD), U21.13 (OUTC), U21.14 (OUTB), U21.9 (GND2); no longer R169.2
- net +3V3: now reaches U20.3 (+3V3)
- net +3V3: now also U21.1 (VDD1)
- net at U1.14 (SER): now also U21.15 (OUTA); no longer R166.2
- new net: R169.2, U21.5 (IND)
- new net: R166.2, U21.2 (INA)
- new net: R167.2, U21.3 (INB)
- new net: R168.2, U21.4 (INC)
- new net: R170.2, U21.6 (INE)
- new net Earth: D1.1, PS1.1 (AC/N)
- new net VAC: D1.2, PS1.2 (AC/L)
- no-connect marks 16 -> 15

Commit message: Update a shit ton
Parts:
- removed NE1, NE10, NE11, NE12, NE13, NE14, NE15, NE16, NE17, NE18, NE2, NE3, NE4, NE5, NE6, NE7, NE8, NE9: INS-1, NixFootprints:INS-1, symbol NixSymbols:INS-1
- removed PS1: IRM-05-5, Converter_ACDC:Converter_ACDC_MeanWell_IRM-05-xx_THT, symbol Converter_ACDC:IRM-05-5
- removed Q151, Q152, Q153, Q154, Q155, Q156, Q157, Q158, Q159, Q160, Q161, Q162, Q163, Q164, Q165, Q166, Q167, Q168: MMBTA42, NixFootprints:SOT-23 No Courtyard, symbol NixMinis:Mini_BJT_NPN
- removed R172, R173, R174, R175, R176, R177, R178, R179, R180, R181, R182, R183, R184, R185, R186, R187, R188: 10K, Resistor_SMD:R_0402_1005Metric, symbol NixMinis:Mini_R
- removed R189, R190, R191, R192, R193, R194, R195, R196, R197, R198, R199, R200, R201, R202, R203, R204, R205, R206: 100K, Resistor_SMD:R_1206_3216Metric, symbol NixMinis:Mini_R
- removed U20: RP2040-Tiny, NixFootprints:RP2040-Tiny Package Extra Clearance SMD, symbol NixSymbols:RP2040-Tiny-Waveshare
- removed U39, U40: 74HC595_Slim, Package_SO:SOIC-16_3.9x9.9mm_P1.27mm, symbol NixSymbols:74HC595_Slim
- added C10, C11, C12, C13, C14, C15, C16, C17, C18, C19, C20, C21, C22, C5, C8, C9: 1uF, Capacitor_THT:C_Radial_D5.0mm_H5.0mm_P2.00mm, symbol NixMinis:Mini_C
- added NE1, NE10, NE11, NE12, NE13, NE14, NE15, NE16, NE17, NE18, NE19, NE2, NE20, NE21, NE22, NE23, NE24, NE3, NE4, NE5, NE6, NE7, NE8, NE9: (no value), FeriNixie:NeonIndicator_A1B_A1C, symbol FeriNixie:NeonIndicator_A1B_A1C
- added PS1, PS2: IRM-02-5, Converter_ACDC:Converter_ACDC_MeanWell_IRM-02-xx_THT, symbol Converter_ACDC:IRM-02-5
- added R16, R17, R18, R19, R20, R31: 100K, Resistor_SMD:R_1206_3216Metric, symbol NixMinis:Mini_R
- added R21, R22, R23, R24, R25, R26, R27, R28, R29, R30: 330, Resistor_SMD:R_0402_1005Metric, symbol NixMinis:Mini_R
- added U38: RP2040-Tiny, NixFootprints:RP2040-Tiny Package Extra Clearance, symbol NixSymbols:RP2040-Tiny-Waveshare
- added U39, U40, U41, U42, U43, U44, U45, U46, U47, U48: GAQY214DE_DEH, Package_DIP:SMDIP-4_W7.62mm, symbol NixSymbols:GAQY214DE_DEH
- renumbered C6 to C1, C5 to C2, C7 to C3, C8 to C4, C1 to C6, C2 to C7, R82 to R100, R83 to R101, R84 to R102, R85 to R103, R86 to R104, R87 to R105, R88 to R106, R89 to R107, R90 to R108, R91 to R109, R92 to R110, R93 to R111, R94 to R112, R95 to R113, R96 to R114, R97 to R115, R98 to R116, R99 to R117, R100 to R118, R101 to R119, R102 to R120, R103 to R121, R104 to R122, R105 to R123, R106 to R124, R107 to R125, R108 to R126, R109 to R127, R110 to R128, R111 to R129, R112 to R130, R113 to R131, R114 to R132, R115 to R133, R116 to R134, R117 to R135, R118 to R136, R119 to R137, R120 to R138, R121 to R139, R122 to R140, R123 to R141, R124 to R142, R125 to R143, R126 to R144, R127 to R145, R128 to R146, R129 to R147, R130 to R148, R131 to R149, R132 to R150, R133 to R151, R134 to R152, R135 to R153, R136 to R154, R137 to R155, R138 to R156, R139 to R157, R140 to R158, R141 to R159, R142 to R160, R143 to R161, R144 to R162, R145 to R163, R146 to R164, R147 to R165, R148 to R166, R149 to R167, R150 to R168, R151 to R169, R152 to R170, R153 to R171, R154 to R172, R155 to R173, R156 to R174, R157 to R175, R158 to R176, R159 to R177, R160 to R178, R161 to R179, R162 to R180, R163 to R181, R164 to R182, R165 to R183, R171 to R184, R166 to R202, R167 to R203, R168 to R204, R169 to R205, R170 to R206, R16 to R34, R17 to R35, R18 to R36, R19 to R37, R20 to R38, R21 to R39, R22 to R40, R23 to R41, R24 to R42, R25 to R43, R26 to R44, R27 to R45, R28 to R46, R29 to R47, R30 to R48, R31 to R49, R32 to R50, R33 to R51, R34 to R52, R35 to R53, R36 to R54, R37 to R55, R38 to R56, R39 to R57, R40 to R58, R41 to R59, R42 to R60, R43 to R61, R44 to R62, R45 to R63, R46 to R64, R47 to R65, R48 to R66, R49 to R67, R50 to R68, R51 to R69, R52 to R70, R53 to R71, R54 to R72, R55 to R73, R56 to R74, R57 to R75, R58 to R76, R59 to R77, R60 to R78, R61 to R79, R62 to R80, R63 to R81, R64 to R82, R65 to R83, R66 to R84, R67 to R85, R68 to R86, R69 to R87, R70 to R88, R71 to R89, R72 to R90, R73 to R91, R74 to R92, R75 to R93, R76 to R94, R77 to R95, R78 to R96, R79 to R97, R80 to R98, R81 to R99, U24 to U1, U33 to U10, U34 to U11, U35 to U12, U36 to U13, U37 to U14, U38 to U15, U1 to U16, U2 to U17, U3 to U18, U4 to U19, U25 to U2, U5 to U20, U6 to U21, U7 to U22, U8 to U23, U9 to U24, U10 to U25, U11 to U26, U12 to U27, U13 to U28, U14 to U29, U26 to U3, U15 to U30, U16 to U31, U17 to U32, U18 to U33, U19 to U34, U21 to U37, U27 to U4, U28 to U5, U29 to U6, U30 to U7, U31 to U8, U32 to U9
Connections:
- net +170V: now also C10.1, C11.1, C12.1, C13.1, C14.1, C15.1, C16.1, C17.1, C18.1, C19.1, C20.1, C21.1, C22.1, C8.1, C9.1
- net +3V3: now also U38.3 (+3V3)
- net +5V: now also C5.2, PS1.4 (+Vo), U38.1 (+5V); no longer C1.2, C2.2, C3.2, C4.2, C6.2, U16.16 (VCC), U17.16 (VCC), U18.16 (VCC), U19.16 (VCC), U20.16 (VCC), U21.16 (VCC), U22.16 (VCC), U23.16 (VCC), U24.16 (VCC), U25.16 (VCC), U31.16 (VCC), U32.16 (VCC), U33.16 (VCC), U34.16 (VCC), U37.16 (VDD2)
- net Earth: now also PS1.1 (AC/N), PS2.1 (AC/N), U42.4, U43.4, U44.4, U45.4, U46.4, U48.4
- net GND: now also C5.1, PS1.3 (-Vo), U38.2 (GND), U39.2, U40.2, U41.2, U42.2, U43.2, U44.2, U45.2, U46.2, U47.2, U48.2; no longer C6.1
- net TBGND: now also C6.1, C10.2, C11.2, C12.2, C13.2, C14.2, C15.2, C16.2, C17.2, C18.2, C19.2, C20.2, C21.2, C22.2, C8.2, C9.2, PS2.3 (-Vo); no longer U16.10 (~{SRCLR}), U16.11 (SRCLK), U16.12 (RCLK), U16.13 (~{OE}), U17.10 (~{SRCLR}), U17.11 (SRCLK), U17.12 (RCLK), U17.13 (~{OE}), U18.10 (~{SRCLR}), U18.11 (SRCLK), U18.12 (RCLK), U18.13 (~{OE}), U19.10 (~{SRCLR}), U19.11 (SRCLK), U19.12 (RCLK), U19.13 (~{OE}), U20.10 (~{SRCLR}), U20.11 (SRCLK), U20.12 (RCLK), U20.13 (~{OE}), U21.10 (~{SRCLR}), U21.11 (SRCLK), U21.12 (RCLK), U21.13 (~{OE}), U22.10 (~{SRCLR}), U22.11 (SRCLK), U22.12 (RCLK), U22.13 (~{OE}), U23.10 (~{SRCLR}), U23.11 (SRCLK), U23.12 (RCLK), U23.13 (~{OE}), U24.10 (~{SRCLR}), U24.11 (SRCLK), U24.12 (RCLK), U24.13 (~{OE}), U25.10 (~{SRCLR}), U25.11 (SRCLK), U25.12 (RCLK), U25.13 (~{OE}), U26.10 (~{SRCLR}), U26.11 (SRCLK), U26.12 (RCLK), U26.13 (~{OE}), U27.10 (~{SRCLR}), U27.11 (SRCLK), U27.12 (RCLK), U27.13 (~{OE}), U28.10 (~{SRCLR}), U28.11 (SRCLK), U28.12 (RCLK), U28.13 (~{OE}), U29.10 (~{SRCLR}), U29.11 (SRCLK), U29.12 (RCLK), U29.13 (~{OE}), U30.10 (~{SRCLR}), U30.11 (SRCLK), U30.12 (RCLK), U30.13 (~{OE}), U31.10 (~{SRCLR}), U31.11 (SRCLK), U31.12 (RCLK), U31.13 (~{OE}), U32.10 (~{SRCLR}), U32.11 (SRCLK), U32.12 (RCLK), U32.13 (~{OE}), U33.10 (~{SRCLR}), U33.11 (SRCLK), U33.12 (RCLK), U33.13 (~{OE}), U34.10 (~{SRCLR}), U34.11 (SRCLK), U34.12 (RCLK), U34.13 (~{OE}), U37.11 (OUTE), U37.12 (OUTD), U37.13 (OUTC), U37.14 (OUTB)
- net VAC: now also PS1.2 (AC/L), PS2.2 (AC/L), U39.3, U40.3, U41.3, U47.3
- net at R205.1: now also U38.20 (3)
- net at R205.2: now also U37.4 (INC); no longer U37.5 (IND)
- net at R206.1: now also U38.19 (4)
- net at R204.1: now also U38.21 (2)
- net at R203.1: now also U38.22 (1)
- net at R202.1: now also U38.23 (0)
- net at U37.10 (OUTF): now also U16.14 (SER)
- net at U37.15 (OUTA): no longer U16.14 (SER)
- net at U37.2 (INA): no longer R202.2
- net at U37.3 (INB): now also R206.2; no longer R203.2
- net at R204.2: now also U37.5 (IND); no longer U37.4 (INC)
- net at U37.6 (INE): now also R203.2; no longer R206.2
- net at U37.7 (INF): now also R202.2
- new net: NE1.1 (A), NE2.1 (A), NE21.1 (A), NE3.1 (A), NE4.1 (A), NE5.1 (A), U39.4
- new net: NE1.2 (K), NE11.2 (K), NE16.2 (K), NE6.2 (K), R16.1
- new net: NE16.1 (A), NE17.1 (A), NE18.1 (A), NE19.1 (A), NE20.1 (A), NE24.1 (A), U47.4
- new net: NE13.2 (K), NE18.2 (K), NE3.2 (K), NE8.2 (K), R18.1
- new net: R16.2, U42.3
- new net: NE12.2 (K), NE17.2 (K), NE2.2 (K), NE7.2 (K), R17.1
- new net: NE11.1 (A), NE12.1 (A), NE13.1 (A), NE14.1 (A), NE15.1 (A), NE23.1 (A), U41.4
- new net: NE21.2 (K), NE22.2 (K), NE23.2 (K), NE24.2 (K), R31.1
- new net: R25.1, U46.1
- new net: R20.2, U46.3
- new net: R27.1, U40.1
- new net: NE10.1 (A), NE22.1 (A), NE6.1 (A), NE7.1 (A), NE8.1 (A), NE9.1 (A), U40.4
- new net: U16.10 (~{SRCLR}), U17.10 (~{SRCLR}), U18.10 (~{SRCLR}), U19.10 (~{SRCLR}), U20.10 (~{SRCLR}), U21.10 (~{SRCLR}), U22.10 (~{SRCLR}), U23.10 (~{SRCLR}), U24.10 (~{SRCLR}), U25.10 (~{SRCLR}), U26.10 (~{SRCLR}), U27.10 (~{SRCLR}), U28.10 (~{SRCLR}), U29.10 (~{SRCLR}), U30.10 (~{SRCLR}), U31.10 (~{SRCLR}), U32.10 (~{SRCLR}), U33.10 (~{SRCLR}), U34.10 (~{SRCLR}), U37.12 (OUTD)
- new net: U16.11 (SRCLK), U17.11 (SRCLK), U18.11 (SRCLK), U19.11 (SRCLK), U20.11 (SRCLK), U21.11 (SRCLK), U22.11 (SRCLK), U23.11 (SRCLK), U24.11 (SRCLK), U25.11 (SRCLK), U26.11 (SRCLK), U27.11 (SRCLK), U28.11 (SRCLK), U29.11 (SRCLK), U30.11 (SRCLK), U31.11 (SRCLK), U32.11 (SRCLK), U33.11 (SRCLK), U34.11 (SRCLK), U37.11 (OUTE)
- new net: U16.12 (RCLK), U17.12 (RCLK), U18.12 (RCLK), U19.12 (RCLK), U20.12 (RCLK), U21.12 (RCLK), U22.12 (RCLK), U23.12 (RCLK), U24.12 (RCLK), U25.12 (RCLK), U26.12 (RCLK), U27.12 (RCLK), U28.12 (RCLK), U29.12 (RCLK), U30.12 (RCLK), U31.12 (RCLK), U32.12 (RCLK), U33.12 (RCLK), U34.12 (RCLK), U37.13 (OUTC)
- new net: U16.13 (~{OE}), U17.13 (~{OE}), U18.13 (~{OE}), U19.13 (~{OE}), U20.13 (~{OE}), U21.13 (~{OE}), U22.13 (~{OE}), U23.13 (~{OE}), U24.13 (~{OE}), U25.13 (~{OE}), U26.13 (~{OE}), U27.13 (~{OE}), U28.13 (~{OE}), U29.13 (~{OE}), U30.13 (~{OE}), U31.13 (~{OE}), U32.13 (~{OE}), U33.13 (~{OE}), U34.13 (~{OE}), U37.14 (OUTB)
- new net: NE14.2 (K), NE19.2 (K), NE4.2 (K), NE9.2 (K), R19.1
- new net: R19.2, U45.3
- new net: R26.1, U39.1
- new net: NE10.2 (K), NE15.2 (K), NE20.2 (K), NE5.2 (K), R20.1
- new net: R22.1, U43.1
- new net: R30.1, U48.1
- new net: R31.2, U48.3
- new net: R23.1, U44.1
- new net: R18.2, U44.3
- new net: R17.2, U43.3
- new net: R29.1, U47.1
- new net: R21.1, U42.1
- new net: R24.1, U45.1
- new net: R28.1, U41.1
- new net +5VISO: C1.2, C2.2, C3.2, C4.2, C6.2, PS2.4 (+Vo), U16.16 (VCC), U17.16 (VCC), U18.16 (VCC), U19.16 (VCC), U20.16 (VCC), U21.16 (VCC), U22.16 (VCC), U23.16 (VCC), U24.16 (VCC), U25.16 (VCC), U31.16 (VCC), U32.16 (VCC), U33.16 (VCC), U34.16 (VCC), U37.16 (VDD2)
- new net H0: R21.2, U38.12 (11)
- new net H1: R22.2, U38.13 (10)
- new net H2: R23.2, U38.14 (9)
- new net H3: R24.2, U38.15 (8)
- new net H4: R25.2, U38.16 (7)
- new net H5: R30.2, U38.17 (6)
- new net V0: R26.2, U38.8 (15)
- new net V1: R27.2, U38.9 (14)
- new net V2: R28.2, U38.10 (13)
- new net V3: R29.2, U38.11 (12)
- no-connect marks 15 -> 5
Other:
- moved on the sheet: U37
